File: schematics/board/BKU.brd (EAGLE design)
At the start: 94 x 94 mm, 68 parts, among them Q1 8MHz, Q2 32,768KHz, U1 STM32F405RGT6

Commit message: Добавлена плата MAG
Connections:
- new net RX-ES: U$13.36, U1.62
- new net TX-ES: U$13.37, U1.29
Changed lines of the file:
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@@
 <?xml version="1.0" encoding="utf-8"?>
 <!DOCTYPE eagle SYSTEM "eagle.dtd">
-<eagle version="9.5.1">
+<eagle version="9.6.0">
 <drawing>
 <settings>
@@
 <via x="11.1" y="80.049" extent="1-16" drill="1"/>
 </signal>
+<signal name="RX-ES">
+<contactref element="U$13" pad="36"/>
+<contactref element="U1" pad="62"/>
+<wire x1="-14.36" y1="16.69" x2="-53.55" y2="17.1" width="0" layer="19" extent="1-1"/>
+</signal>
+<signal name="TX-ES">
+<contactref element="U$13" pad="37"/>
+<contactref element="U1" pad="29"/>
+<wire x1="-14.36" y1="17.96" x2="-48.55" y2="5.76" width="0" layer="19" extent="1-1"/>
+</signal>
 </signals>

Commit message: Исправлены компоненты
Parts:
- removed R28, R29, R30, R31, R32: 3.3, resistor-shunt:SMK
- added MAG: (no value), pinheadCS:1X04
- added R15: 2k, resistor:R0603
- added R21, R22, R23, R24: 3k3, resistor:R0603
- added R25, R26: 5k1, resistor:R0603
- Q2: device 9C-8.000MEEJ-T:XTAL_9C-8.000MEEJ-T -> CanCubeSat:C005R
- R1, R14, R3, R4: device resistor-shunt:BVS -> resistor:R0603
- R16: value 1M -> 2k; device resistor-shunt:BVS -> resistor:R0603
- R17: value 2k -> 1M; device resistor-shunt:BVS -> resistor:R0603
- R18: value 2k -> 3k3; device resistor-shunt:BVS -> resistor:R0603
- moved D4 205.1 mm to (-82.0, -110.0)
- moved C2 184.1 mm to (-84.0, -100.0)
- moved R16 166.3 mm to (-84.0, -105.0)
- moved U$1 144.4 mm to (59.2, 55.6)
- moved R4 137.2 mm to (-84.0, -65.0)
- moved R14 136.8 mm to (-84.0, -70.0)
- moved U$12 134.3 mm to (59.0, 18.4)
- moved R18 132.3 mm to (-84.0, -75.0)
- moved U$4 128.5 mm to (66.4, 71.3)
- moved U$9 127.3 mm to (72.0, 5.40)
- moved U$10 124.5 mm to (63.8, 12.6)
- moved U$20 123.4 mm to (70.1, 23.4)
- moved U$6 123.3 mm to (47.4, 73.1)
- moved U$11 121.6 mm to (59.0, 35.1)
- moved BSK3 119.1 mm to (86.6, 47.0), turned to 90 degrees
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Connections:
- new net SCL: MAG.3, R25.2, U1.29
- new net SDA: MAG.4, R26.2, U1.30
- new net TIME-ES: U$13.5
- new net TIME-G: U$1.PPS
- net DAT0: now also R23.2; no longer R29.1
- net DAT1: now also R24.2; no longer R30.1
- net GND: now also MAG.1, R16.1; no longer R18.1, U$13.32
- net MTCK: now also R21.2; no longer R31.1
- net MTDI: now also R18.2; no longer R32.1
- net MTDO: now also R22.2; no longer R28.1
- net N$11: now also R14.1; no longer R14.2
- net N$12: now also R4.1; no longer R4.2
- net N$15: now also R17.1; no longer R16.2
- net N$30: now also R17.2; no longer R16.1
- net N$34: now also Q2.P$2; no longer Q2.2
- net N$35: now also Q2.P$1; no longer Q2.1
- net N$37: now also R15.2; no longer R17.1
- net N$38: now also R15.1; no longer R17.2
- net N$40: now also R16.2; no longer R18.2
- net RX-ES: now also U1.42; no longer U1.62
- net RX-S: now also U1.51
- net SWC: now also R3.1; no longer R3.2
- net SWD: now also R1.1; no longer R1.2
- net TX-ES: now also U1.43; no longer U1.29
- net TX-S: now also U1.52
- net VDD: now also MAG.2, R1.2, R14.2, R18.1, R21.1, R22.1, R23.1, R24.1, R25.1, R26.1, R3.2, R4.2; no longer R1.1, R14.1, R28.2, R29.2, R3.1, R30.2, R31.2, R32.2, R4.1

Commit message: Незначительные изменения БКУ
Parts:
- removed C13, C9: 47µ, rcl:C1206
- removed D3, D4: (no value), display-hp:HLMP6
- removed U$3: CD, untitled:CD
- added C12: 0,1µ, rcl:C0603
- added C17: 47µ, rcl:C1206
- added LED-B#2, LED-G#2, LED2, LED3: (no value), led:CHIPLED_0603
- added R27, R28: 2k, resistor:R0603
- added U$14: SD, CanCubeSat:SD
- C16: value 0.1u -> 47µ; device rcl:C025-024X044 -> rcl:C1206
- U$1: value NEO -> GPS; device untitled:NEO -> CanCubeSat:GPS
- moved C16 197.9 mm to (-75.0, -142.0)
- moved R11 134.2 mm to (78.1, 66.4), turned to 180 degrees
- moved R19 128.9 mm to (78.1, 68.5), turned to 180 degrees
- moved R10 124.6 mm to (78.2, 64.3), turned to 180 degrees
- moved U$7 124.2 mm to (45.0, 80.4)
- moved R20 105.1 mm to (78.1, 62.2), turned to 180 degrees
- moved U$5 104.7 mm to (69.1, 57.7)
- moved U$4 78.2 mm to (0.00, 30.0), turned to 270 degrees
- moved U$9 60.1 mm to (75.0, 65.4)
- moved U$6 48.3 mm to (0.00, 64.0), turned to 270 degrees
- moved U$19 47.0 mm to (32.9, 11.9)
- moved JTAG 38.8 mm to (29.4, 67.6)
- moved U$1 38.5 mm to (25.4, 37.2), turned to 90 degrees
- moved U$20 24.6 mm to (79.6, 46.1), turned to 90 degrees
- moved U$18 24.6 mm to (69.7, 82.4), turned to 180 degrees
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Connections:
- removed net N$36: C13.1, C9.2
- new net GND2: R27.2
- new net N$50: LED-B#2.A
- new net N$51: LED-B#2.C, R27.1
- new net N$52: LED-G#2.C, R28.2
- net 5V: now also R28.1
- net B2_KEM+: now also U$19.6; no longer U$18.6
- net B2_KEM-: now also U$19.7; no longer U$18.7
- net B2_KHEAT: now also U$19.5; no longer U$18.5
- net B2_KVCC: now also U$19.4; no longer U$18.4
- net B4_KEM+: now also U$18.6; no longer U$19.6
- net B4_KEM-: now also U$18.7; no longer U$19.7
- net B4_KHEAT: now also U$18.5; no longer U$19.5
- net B4_KVCC: now also U$18.4; no longer U$19.4
- net BUS+: now also C16.1, C17.1; no longer C9.1
- net BUS-: now also LED-G#2.A
- net DAT0: now also U$14.DAT0; no longer U$3.DAT0
- net DAT1: now also U$14.DAT1; no longer U$3.DAT1
- net GND: now also C12.1, C16.2, C17.2, U$14.VDD; no longer C13.2, C16.1, U$3.VDD
- net MTCK: now also U$14.DAT3; no longer U$3.CD/DAT3
- net MTDI: now also U$14.DAT2; no longer U$3.DAT2
- net MTDO: now also U$14.CMD; no longer U$3.CMD
- net MTMS: now also U$14.CLK; no longer U$3.CLK
- net N$37: now also LED2.C; no longer D3.K
- net N$40: now also LED3.C; no longer D4.K
- net VDD: now also C12.2, LED2.A, LED3.A, U$14.VSS; no longer C16.2, D3.A, D4.A, U$3.VSS
Other:
- outline, holes or cut-outs redrawn

Commit message: Добавлена плата RADIO
Parts:
- removed U$1: GPS, CanCubeSat:GPS
- removed U$2: RADIO, untitled:RADIO
- added GPS: GPS, CanCubeSat:GPS
- added R29: 10k, resistor:R0603
- added RADIO: RADIO, CanCubeSat:RADIO
- moved C17 228.7 mm to (68.1, 20.7), turned to 270 degrees
- moved C16 224.4 mm to (79.5, 20.7), turned to 270 degrees
- moved R8 164.0 mm to (70.2, 20.6), turned to 270 degrees
- moved C14 156.7 mm to (73.8, 20.1), turned to 180 degrees
- moved C6 154.4 mm to (68.8, 32.3)
- moved R12 148.9 mm to (80.6, 28.1), turned to 180 degrees
- moved R13 141.9 mm to (66.8, 28.1)
- moved C5 120.0 mm to (72.6, 31.8), turned to 270 degrees
- moved C1 117.7 mm to (75.0, 31.8), turned to 90 degrees
- moved R9 117.6 mm to (77.4, 20.6), turned to 270 degrees
- moved C15 108.4 mm to (78.8, 32.3), turned to 180 degrees
- moved U$12 33.9 mm to (78.8, 30.1)
- moved U$13 29.0 mm to (47.5, 74.5), turned to 90 degrees
- moved U$7 23.3 mm to (55.0, 59.4)
- moved LED-B#2 23.3 mm to (48.6, 59.1)
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- renumbered U$14 to SD
Connections:
- new net AUX: RADIO.P$5, U$13.4
- net GND: now also GPS.GND, R29.2, RADIO.P$1, RADIO.P$15, RADIO.P$16, RADIO.P$17, RADIO.P$7, RADIO.P$9; no longer U$1.GND, U$2.GND
- net M1: now also R29.1, RADIO.P$2; no longer U$2.M1
- net N$41: now also GPS.RX; no longer U$1.RX
- net N$42: now also GPS.TX; no longer U$1.TX
- net RX-R: now also RADIO.P$4; no longer U$2.TXD
- net TIME-G: now also GPS.PPS; no longer U$1.PPS
- net TX-R: now also RADIO.P$3; no longer U$2.RXD
- net VDD: now also GPS.UCC, RADIO.P$6; no longer U$1.UCC, U$2.VCC

Commit message: Пытаем плату БКУ компоновкой
Parts:
- removed JP1: (no value), pinhead:1X04
- removed LED-G#2: (no value), led:CHIPLED_0603
- removed R10, R11, R14, R4: 10k, resistor:R0603
- removed R19: 1M, resistor:R0603
- removed R20: 510k, resistor:R0603
- removed R28: 2k, resistor:R0603
- removed U$9: FS8205A+, CanCubeSat:FS8205A+
- moved RADIO 221.5 mm to (80.2, 43.0)
- moved C8 110.3 mm to (30.0, 56.8)
- moved C10 106.4 mm to (13.2, 37.7), turned to 90 degrees
- moved C7 104.4 mm to (29.9, 54.8)
- moved MAG 81.6 mm to (-18.0, 49.0)
- moved U1 78.5 mm to (18.6, 48.2), turned to 90 degrees
- moved C11 61.4 mm to (19.6, 37.7), turned to 90 degrees
- moved Q1 58.1 mm to (36.5, 48.6), turned to 270 degrees
- moved U$13 55.2 mm to (24.0, 24.5), turned to 270 degrees
- moved JTAG 45.5 mm to (-17.4, 58.1)
- moved GPS 36.7 mm to (33.7, 71.0), turned to 0 degrees
- moved U$8 36.0 mm to (104.3, 44.4)
- moved U$4 34.0 mm to (0.00, 64.0)
- moved U$6 34.0 mm to (0.00, 30.0)
- moved Q2 28.0 mm to (16.0, 38.1)
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Connections:
- removed net 3V3: U$4.3V3/BUS0, U$4.3V3/BUS1
- removed net B1_KVCC: R10.1, R11.1, R19.1, R20.1, U$18.15
- removed net BUS-: LED-G#2.A, R20.2, U$9.23
- removed net GND2: R27.2
- removed net N$1: JP1.4, U1.22
- removed net N$10: JP1.3, U1.23
- removed net N$11: R14.1, U1.50
- removed net N$12: R4.1, U1.55
- removed net N$16: JP1.1, U1.20
- removed net N$2: JP1.2, U1.21
- removed net N$50: LED-B#2.A
- removed net N$52: LED-G#2.C, R28.2
- removed net N$8: R10.2, U$9.4
- removed net N$9: R11.2, U$9.5
- net 5V: no longer R28.1
- net BUS+: no longer R19.2
- net GND: now also R27.2; no longer U$9.67, U$9.HEAT
- net N$3: now also LED-B#2.A
- net VDD: now also U$4.3V3/BUS0, U$4.3V3/BUS1; no longer R14.2, R4.2

Commit message: Изменения в компоновке БКУ
Parts:
- moved R29 250.8 mm to (55.0, 41.8)
- moved LED3 217.7 mm to (72.5, 15.4), turned to 270 degrees
- moved R26 209.9 mm to (75.5, 17.5)
- moved R25 208.1 mm to (75.5, 19.6)
- moved LED2 203.3 mm to (13.5, 47.9), turned to 90 degrees
- moved R16 198.7 mm to (72.4, 17.5)
- moved C2 196.9 mm to (72.4, 19.6), turned to 180 degrees
- moved C12 190.1 mm to (45.4, 15.2)
- moved R24 169.7 mm to (48.5, 11.0)
- moved R23 167.9 mm to (48.5, 13.1)
- moved R22 166.1 mm to (48.5, 15.2)
- moved R21 159.4 mm to (45.4, 13.1), turned to 180 degrees
- moved R18 155.4 mm to (45.4, 11.0), turned to 180 degrees
- moved R17 151.3 mm to (32.1, 52.0)
- moved R3 148.6 mm to (13.5, 52.1), turned to 180 degrees
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Routing:
- net GND: track 0.00 -> 319.5 mm, vias 0 -> 2
- net BUS+: track 0.00 -> 295.8 mm, vias 0 -> 9
- net N$24: track 0.00 -> 29.2 mm, vias 0 -> 2
- net N$39: track 0.00 -> 14.7 mm, vias 0 -> 2
- net N$25: track 0.00 -> 14.4 mm, vias 0 -> 2
- net VDD: track 0.00 -> 6.34 mm
- net 5V: track 0.00 -> 6.21 mm
- net N$28: track 0.00 -> 6.06 mm
- net N$33: track 0.00 -> 5.79 mm
- net N$32: track 0.00 -> 2.66 mm
- net N$31: track 0.00 -> 2.64 mm
- added copper zone on layer 1, net GND
- removed copper zone on layer 1, net GND1

Commit message: Изменения в БКУ
Parts:
- GPS: value GPS -> GPSNEO6M; device CanCubeSat:GPS -> CanCubeSat:GPS-NEO6M
- JTAG: device pinheadCS:1X04 -> pinheadCS:1X06
- moved LED2 3.54 mm to (13.0, 51.4)
- moved R1 3.54 mm to (13.0, 57.8)
- moved R15 3.54 mm to (13.0, 53.5)
- moved R3 3.54 mm to (13.0, 55.6)
- moved U1 3.54 mm to (22.1, 51.7)
- moved C10 3.50 mm to (13.8, 41.3)
- moved C11 3.50 mm to (18.5, 41.3)
- moved Q2 3.50 mm to (16.1, 41.4)
- moved R7 3.50 mm to (20.6, 41.3)
- moved C1 1.68 mm to (60.9, 36.2)
- moved C16 1.68 mm to (65.3, 24.9)
- moved R13 1.68 mm to (52.7, 32.5)
- moved U$11 1.68 mm to (54.6, 34.6)
- moved U$12 1.68 mm to (64.6, 34.6)
- moved C14 1.68 mm to (59.6, 24.3)
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Connections:
- removed net VSS: U1.18, U1.63
- net GND: now also GPS.P$4, JTAG.1, U1.18, U1.28, U1.60, U1.63; no longer GPS.GND
- net MTCK: now also JTAG.5; no longer JTAG.3
- net MTDI: now also JTAG.6; no longer JTAG.4
- net MTDO: now also JTAG.3; no longer JTAG.1
- net MTMS: now also JTAG.4; no longer JTAG.2
- net N$41: now also GPS.P$2; no longer GPS.RX
- net N$42: now also GPS.P$3; no longer GPS.TX
- net TIME-G: now also GPS.P$1; no longer GPS.PPS
- net VDD: now also GPS.P$5, JTAG.2; no longer GPS.UCC

Commit message: Изменения в БКУ
Connections:
- removed net VDDA: U1.13
- removed net VSSA: U1.12
- net GND: now also U1.12
- net VDD: now also U1.13
