File: schematics/board/BKU.brd (EAGLE design)
At the start: 94 x 94 mm, 73 parts, among them Q1 8MHz, Q2 32,768KHz, U1 STM32F405RGT6

Commit message: Незначительные изменения БКУ
Parts:
- C7, C8: value 54pF -> 27pF
Changed lines of the file:
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@@
 <attribute name="VALUE" x="53.35" y="34.19" size="1.27" layer="27"/>
 </element>
-<element name="C7" library="rcl" library_urn="urn:adsk.eagle:library:334" package="C0603" package3d_urn="urn:adsk.eagle:package:23616/2" value="54pF" x="32.08" y="54.13" smashed="yes">
+<element name="C7" library="rcl" library_urn="urn:adsk.eagle:library:334" package="C0603" package3d_urn="urn:adsk.eagle:package:23616/2" value="27pF" x="32.08" y="54.13" smashed="yes">
 <attribute name="POPULARITY" value="73" x="103.2" y="-27.15" size="1.778" layer="27" display="off"/>
 <attribute name="SPICEPREFIX" value="C" x="103.2" y="-27.15" size="1.778" layer="27" display="off"/>
 <attribute name="VALUE" x="31.445" y="52.225" size="1.27" layer="27"/>
 </element>
-<element name="C8" library="rcl" library_urn="urn:adsk.eagle:library:334" package="C0603" package3d_urn="urn:adsk.eagle:package:23616/2" value="54pF" x="32.03" y="56.28" smashed="yes">
+<element name="C8" library="rcl" library_urn="urn:adsk.eagle:library:334" package="C0603" package3d_urn="urn:adsk.eagle:package:23616/2" value="27pF" x="32.03" y="56.28" smashed="yes">
 <attribute name="POPULARITY" value="73" x="109.5" y="-25" size="1.778" layer="27" display="off"/>
 <attribute name="SPICEPREFIX" value="C" x="109.5" y="-25" size="1.778" layer="27" display="off"/>

Commit message: Доработана плата БКУ
Parts:
- moved MAG 2.97 mm to (74.8, 24.9), flipped to the bottom, turned to 180 degrees
- moved U$8 0.85 mm to (75.8, 34.8)
Connections:
- new net N$6: U1.54, U1.58
- net TIME-ES: now also U1.22; no longer U1.15
- net TIME-G: now also U1.23, U1.59
Routing:
- net TIME-G: track 29.5 -> 45.0 mm, vias 1 -> 3
- net SDA: track 87.8 -> 96.0 mm
- net SCL: track 79.9 -> 87.6 mm
- net TIME-ES: track 21.1 -> 28.1 mm
- net B3_KHEAT: track 42.6 -> 49.2 mm
- net VDD: track 450.2 -> 456.1 mm, vias 24 -> 25
- net AUX: track 56.3 -> 61.5 mm
- net 5V: track 292.6 -> 297.3 mm
- net B5_KHEAT: track 48.8 -> 52.9 mm
- net N$6: track 0.00 -> 3.77 mm
- net B2A_KEM+: track 127.3 -> 130.1 mm
- net B5_KEM+: track 22.5 -> 23.7 mm
- net SHCP: track 164.5 -> 165.6 mm
- net B1_KEM-: track 65.2 -> 66.2 mm
- net I2CINT: track 98.0 -> 98.9 mm
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
Commit message: Изменения в подключении мк
Parts:
- added C13, C9: 2,2µ, rcl:C0603
- added C18, C20, C53, C54, C55: 100nF, rcl:C0603
- added C19: 10µ, rcl:C1206
- moved GPS 1.15 mm to (31.0, 72.3)
- moved LED2 0.65 mm to (12.8, 50.8)
- moved R1 0.60 mm to (12.6, 57.4)
- moved R3 0.54 mm to (12.6, 55.3)
- moved R15 0.54 mm to (12.6, 53.2)
- moved C7 0.45 mm to (32.5, 54.1)
- moved C8 0.45 mm to (32.5, 56.3)
- moved R17 0.45 mm to (32.5, 52.0)
- moved R14 0.40 mm to (9.95, 51.5)
- moved Q1 0.38 mm to (36.8, 48.4)
- moved U1 0.35 mm to (22.1, 51.4)
Connections:
- removed net VCAP_1: U1.31
- removed net VCAP_2: U1.47
- new net N$7: C9.2, U1.31
- new net N$8: C13.2, U1.47
- net GND: now also C13.1, C18.1, C19.1, C20.1, C53.1, C54.1, C55.1, C9.1
- net VDD: now also C18.2, C19.2, C20.2, C53.2, C54.2, C55.2
Routing:
- net GND: track 460.7 -> 530.7 mm, vias 24 -> 28
- net VDD: track 456.1 -> 466.6 mm
- net N$7: track 0.00 -> 10.2 mm, vias 0 -> 2
- net N$41: track 34.6 -> 38.5 mm
- net SWD: track 19.4 -> 23.0 mm
- net SCL: track 87.6 -> 91.1 mm, vias 8 -> 10
- net AUX: track 61.5 -> 58.2 mm
- net N$15: track 39.0 -> 41.6 mm
- net N$8: track 0.00 -> 2.56 mm
- net 5V: track 297.3 -> 299.4 mm
- net SDATM: track 108.4 -> 110.2 mm
- net SWC: track 15.4 -> 17.2 mm
- net N$42: track 37.6 -> 39.1 mm
- net RX-S: track 28.9 -> 30.2 mm
- net DS: track 122.2 -> 123.4 mm
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
Commit message: Обновлены герберы плат
Routing:
- net GND: track 530.7 -> 525.3 mm
Changed lines of the file:
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@@
 <param name="mvStopFrame" value="1"/>
 <param name="mvCreamFrame" value="0"/>
-<param name="mlMinStopFrame" value="4mil"/>
-<param name="mlMaxStopFrame" value="4mil"/>
+<param name="mlMinStopFrame" value="2mil"/>
+<param name="mlMaxStopFrame" value="2mil"/>
 <param name="mlMinCreamFrame" value="0mil"/>
 <param name="mlMaxCreamFrame" value="0mil"/>
@@
 <contactref element="JTAG" pad="1"/>
 <contactref element="BT1" pad="-"/>
-<wire x1="17.575" y1="48.1" x2="16.4" y2="48.1" width="0.2" layer="1"/>
-<wire x1="17.725" y1="49.6" x2="16.4" y2="49.6" width="0.2" layer="1"/>
 <wire x1="8.4718" y1="68.5718" x2="9.487675" y2="68.5718" width="0.3" layer="1"/>
 <via x="9.487675" y="68.5718" extent="1-16" drill="0.35"/>
@@
 <via x="8.5" y="60.5" extent="1-16" drill="0.35"/>
 <wire x1="23.82" y1="45.68" x2="23.82" y2="47.32" width="0.3" layer="1"/>
-<wire x1="23.82" y1="47.32" x2="24" y2="47.5" width="0.3" layer="1"/>
 <wire x1="27.74" y1="48.1" x2="26.1" y2="48.1" width="0.3" layer="1"/>
-<wire x1="26.1" y1="48.1" x2="26" y2="48" width="0.3" layer="1"/>
 <wire x1="33.33" y1="56.28" x2="38.05" y2="61" width="0.3" layer="1"/>
 <wire x1="38.05" y1="61" x2="38.5" y2="61" width="0.3" layer="1"/>
@@
 <wire x1="35.70060625" y1="6.288" x2="36.302" y2="6.88939375" width="0.3" layer="1"/>
 <wire x1="30.11" y1="7.4" x2="30.90739375" y2="7.4" width="0.3" layer="1"/>
-<wire x1="36.302" y1="8.302" x2="37" y2="9" width="0.3" layer="1"/>
 <wire x1="30.90739375" y1="7.4" x2="32.01939375" y2="6.288" width="0.3" layer="1"/>
 <wire x1="36.302" y1="6.88939375" x2="36.302" y2="8.302" width="0.3" layer="1"/>
@@
 <wire x1="75.77895625" y1="10.75" x2="75.75119375" y2="10.7777625" width="0.3" layer="1"/>
 <wire x1="75.75119375" y1="10.7777625" x2="75.7222375" y2="10.7777625" width="0.3" layer="1"/>
-<wire x1="75.7222375" y1="10.7777625" x2="75" y2="11.5" width="0.3" layer="1"/>
 <via x="93.1738" y="31" extent="1-16" drill="0.35"/>
 <wire x1="83.3" y1="23" x2="83.3" y2="23.92016875" width="0.3" layer="1"/>
@@
 <wire x1="83.74" y1="71.76" x2="83.5" y2="72" width="0.3" layer="1"/>
 <wire x1="27.74" y1="53.1" x2="26.8" y2="53.1" width="0.3" layer="1"/>
-<wire x1="26.8" y1="53.1" x2="26.45" y2="52.75" width="0.3" layer="1"/>
 <contactref element="R14" pad="2"/>
 <contactref element="C9" pad="1"/>
