File: schematics/board/HEAT.brd (EAGLE design)
At the start: 12 x 17 mm, 0 parts

Commit message: Создана плата HEAT
Parts:
- added U$1, U$2: PAD, CanCubeSat:PAD
Connections:
- new net N$1: U$1.P$1, U$2.P$1
Routing:
- net N$1: track 0.00 -> 2905.1 mm, vias 0 -> 7
