File: schematics/board/SP.brd (EAGLE design)
At the start: 207.1 x 206.5 mm, 33 parts

Commit message: Плата СБ
Parts:
- added S1: (no value), CanCubeSat:255SB
- added U$1, U$2, U$20, U$21: KCONNECT--, CanCubeSat:KCONNECT-3
- added U$18, U$3, U$4: KCONNECT4, CanCubeSat:KCONNECT-4
- added U$19: KCONNECT1, CanCubeSat:KCONNECT-1
- moved D25 79.7 mm to (50.0, 6.00)
- moved D34 66.8 mm to (72.0, 46.0)
- moved D37 63.1 mm to (31.0, 76.0), turned to 180 degrees
- moved D32 52.4 mm to (10.0, 56.0)
- moved D35 47.4 mm to (50.0, 66.0), turned to 180 degrees
- moved D33 45.8 mm to (72.0, 56.0)
- moved D36 45.4 mm to (50.0, 76.0)
- moved D29 45.2 mm to (31.0, 6.00)
- moved D28 38.8 mm to (10.0, 26.0)
- moved D27 38.1 mm to (72.0, 26.0), turned to 180 degrees
- moved D38 35.8 mm to (31.0, 66.0)
- moved D30 29.2 mm to (10.0, 36.0)
- moved D24 23.8 mm to (50.0, 16.0)
- moved D26 23.7 mm to (72.0, 36.0), turned to 180 degrees
- moved D31 22.4 mm to (10.0, 46.0)
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Connections:
- removed net N$17: D24.C
- removed net N$18: D25.A
- removed net N$20: D26.A
- removed net N$23: D27.C
- removed net N$24: D28.A
- removed net N$26: D29.A
- removed net N$27: D29.C
- removed net N$29: SOL1.IN
- removed net N$30: D1.C, SOL16.OUT
- removed net N$31: D31.C
- removed net N$32: D32.A
- removed net N$33: D32.C
- removed net N$34: D33.A
- removed net N$35: D33.C
- removed net N$36: D34.A
- removed net N$37: D34.C
- removed net N$38: D35.A
- removed net N$39: D35.C
- removed net N$40: D36.A
- removed net N$41: D36.C
- removed net N$42: D37.A
- removed net N$43: D37.C
- removed net N$44: D38.A
- removed net N$45: D1.A, D38.C
- new net BUS+1: D1.A, D1.C, D38.C, U$1.1, U$1.2, U$1.4, U$18.1, U$18.2, U$18.3, U$20.1, U$20.2, U$20.4, U$3.1, U$3.2, U$3.3
- new net BUS-1: D29.A, S1.3, SOL1.IN
- new net N$2: S1.2, U$19.2, U$19.3, U$19.4, U$2.1, U$2.2, U$2.4, U$21.1, U$21.2, U$21.4, U$4.1, U$4.2, U$4.3
- net N$1: now also D29.C; no longer SOL1.OUT
- net N$10: now also D32.C, D33.A; no longer SOL10.OUT
- net N$11: now also D33.C, D34.A; no longer SOL11.OUT
- net N$12: now also D34.C, D35.A; no longer SOL12.OUT
- net N$13: now also D35.C, D36.A; no longer SOL13.OUT
- net N$14: now also D36.C, D37.A; no longer SOL14.OUT
- net N$15: now also D37.C, D38.A; no longer SOL15.OUT
- net N$16: no longer SOL2.OUT
- net N$19: now also D26.A; no longer SOL4.OUT
- net N$22: no longer SOL5.OUT
- net N$28: no longer SOL7.OUT
- net N$3: now also D24.C, D25.A; no longer SOL3.OUT
- net N$6: now also D27.C, D28.A; no longer SOL6.OUT
- net N$8: no longer SOL8.OUT
- net N$9: now also D31.C, D32.A; no longer SOL9.OUT
Routing:
- net BUS+1: track 0.00 -> 184.1 mm
- net N$2: track 0.00 -> 153.5 mm
- net N$10: track 0.00 -> 73.0 mm, vias 0 -> 1
- net BUS-1: track 0.00 -> 69.6 mm
- net N$6: track 0.00 -> 66.1 mm, vias 0 -> 2
- net N$12: track 0.00 -> 53.9 mm, vias 0 -> 1
- net N$19: track 0.00 -> 43.3 mm, vias 0 -> 1
- net N$22: track 0.00 -> 33.5 mm, vias 0 -> 1
- net N$3: track 0.00 -> 28.0 mm, vias 0 -> 1
- net N$9: track 0.00 -> 26.6 mm, vias 0 -> 1
- net N$14: track 0.00 -> 25.1 mm, vias 0 -> 1
- net N$15: track 0.00 -> 24.4 mm, vias 0 -> 1
- net N$16: track 0.00 -> 20.4 mm, vias 0 -> 1
- net N$13: track 0.00 -> 17.6 mm, vias 0 -> 1
- net N$1: track 0.00 -> 17.6 mm, vias 0 -> 1
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
Commit message: Плата СБ готовая
Other:
- board size 207.1 x 206.5 mm -> 82 x 82 mm
Changed lines of the file:
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@@
 <board>
 <plain>
-<wire x1="-40.6" y1="-19.9" x2="136.31" y2="-13.6" width="0" layer="20"/>
-<wire x1="136.31" y1="-13.6" x2="166.51" y2="186.63" width="0" layer="20"/>
-<wire x1="166.51" y1="186.63" x2="-10.4" y2="139.33" width="0" layer="20"/>
-<wire x1="-10.4" y1="139.33" x2="-40.6" y2="-19.9" width="0" layer="20"/>
 <wire x1="7" y1="-9" x2="15" y2="-9" width="0.1" layer="39"/>
 <wire x1="15" y1="-9" x2="15" y2="7.27193125" width="0.1" layer="39"/>
@@
 <wire x1="34.26748125" y1="24.306490625" x2="28.8618" y2="23.204940625" width="0.1" layer="39" curve="66.964296"/>
 <wire x1="23.204940625" y1="28.8618" x2="24.306490625" y2="34.26748125" width="0.1" layer="39" curve="66.964381"/>
+<wire x1="0" y1="0" x2="82" y2="0" width="0.1524" layer="20"/>
+<wire x1="0" y1="82" x2="0" y2="73.6" width="0.1524" layer="20"/>
+<wire x1="0" y1="68.4" x2="0" y2="33.7" width="0.1524" layer="20"/>
+<wire x1="0" y1="28.5" x2="0" y2="0" width="0.1524" layer="20"/>
+<wire x1="82" y1="0" x2="82" y2="8.5" width="0.1524" layer="20"/>
+<wire x1="82" y1="13.7" x2="82" y2="48.5" width="0.1524" layer="20"/>
+<wire x1="82" y1="53.7" x2="82" y2="82" width="0.1524" layer="20"/>
+<wire x1="82" y1="82" x2="0" y2="82" width="0.1524" layer="20"/>
+<wire x1="82" y1="13.7" x2="77.9" y2="13.7" width="0.1524" layer="20"/>
+<wire x1="77.9" y1="13.7" x2="77.9" y2="8.5" width="0.1524" layer="20"/>
+<wire x1="77.9" y1="8.5" x2="82" y2="8.5" width="0.1524" layer="20"/>
+<wire x1="82" y1="53.7" x2="77.9" y2="53.7" width="0.1524" layer="20"/>
+<wire x1="77.9" y1="53.7" x2="77.9" y2="48.5" width="0.1524" layer="20"/>
+<wire x1="77.9" y1="48.5" x2="81.8" y2="48.5" width="0.1524" layer="20"/>
+<wire x1="0" y1="68.4" x2="4.1" y2="68.4" width="0.1524" layer="20"/>
+<wire x1="4.1" y1="68.4" x2="4.1" y2="73.6" width="0.1524" layer="20"/>
+<wire x1="4.1" y1="73.6" x2="0" y2="73.6" width="0.1524" layer="20"/>
+<wire x1="0" y1="28.5" x2="4.2" y2="28.5" width="0.1524" layer="20"/>
+<wire x1="4.2" y1="28.5" x2="4.2" y2="33.7" width="0.1524" layer="20"/>
+<wire x1="4.2" y1="33.7" x2="0" y2="33.7" width="0.1524" layer="20"/>
+<wire x1="81.8" y1="48.5" x2="82" y2="48.5" width="0.1524" layer="20"/>
 </plain>
 <attributes>

Commit message: Плата SP
Routing:
- net N$4: track 0.00 -> 5.59 mm
Changed lines of the file:
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@@
 <wire x1="25" y1="20.5" x2="24.386446875" y2="20.143803125" width="0.5" layer="1"/>
+</signal>
+<signal name="N$4">
+<wire x1="0.1" y1="4.1" x2="0.1" y2="3.6" width="0.1524" layer="1"/>
+<wire x1="0.1" y1="3.6" x2="3.7" y2="0" width="0.1524" layer="1"/>
 </signal>
 </signals>

Commit message: Плата СБ
Parts:
- added LED1: LAP4-BOTTOM, led:P47F-BOTTOM
- added R1: 2k7, rcl:R0603
- SOL1, SOL10, SOL11, SOL13, SOL14, SOL15, SOL2, SOL3, SOL5, SOL6, SOL7, SOL9: value SOLAR -> SOLAR_0
- SOL12, SOL16, SOL4, SOL8: value SOLARSOLAR_1 -> SOLAR_1
- U$1, U$2, U$20, U$21: value KCONNECT-- -> KCONNECT3
- moved S1 0.80 mm to (21.0, 3.00), flipped to the bottom
- moved SOL1 0.79 mm to (11.0, 10.2)
- moved SOL13 0.79 mm to (71.0, 71.8)
- moved SOL14 0.79 mm to (51.0, 71.8)
- moved SOL15 0.79 mm to (31.0, 71.8)
- moved SOL16 0.79 mm to (11.0, 71.8)
- moved SOL2 0.79 mm to (31.0, 10.2)
- moved SOL3 0.79 mm to (51.0, 10.2)
- moved SOL4 0.79 mm to (71.0, 10.2)
- moved SOL10 0.35 mm to (31.0, 51.2)
- moved SOL11 0.35 mm to (51.0, 51.2)
- moved SOL12 0.35 mm to (71.0, 51.2)
- moved SOL5 0.35 mm to (71.0, 30.8)
- moved SOL6 0.35 mm to (51.0, 30.8)
- moved SOL7 0.35 mm to (31.0, 30.8)
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Connections:
- new net N$4: D1.A, D38.C, SOL16.OUT
- new net N$5: LED1.A, R1.1
- net BUS+1: now also R1.2; no longer D1.A, D38.C
- net N$1: now also SOL1.OUT
- net N$10: now also SOL10.OUT
- net N$11: now also SOL11.OUT
- net N$12: now also SOL12.OUT
- net N$13: now also SOL13.OUT
- net N$14: now also SOL14.OUT
- net N$15: now also SOL15.OUT
- net N$16: now also SOL2.OUT
- net N$19: now also SOL4.OUT
- net N$2: now also LED1.C
- net N$22: now also SOL5.OUT
- net N$28: now also SOL7.OUT
- net N$3: now also SOL3.OUT
- net N$6: now also SOL6.OUT
- net N$8: now also SOL8.OUT
- net N$9: now also SOL9.OUT
Routing:
- net BUS-1: track 69.6 -> 26.5 mm
- net N$4: track 5.59 -> 36.8 mm
- net N$2: track 153.5 -> 167.1 mm
- net N$11: track 16.6 -> 28.8 mm, vias 1 -> 0
- net N$28: track 16.6 -> 28.7 mm, vias 1 -> 0
- net N$13: track 17.6 -> 29.2 mm, vias 1 -> 0
- net N$8: track 17.4 -> 28.6 mm
- net N$1: track 17.6 -> 28.3 mm, vias 1 -> 0
- net BUS+1: track 184.1 -> 194.5 mm
- net N$19: track 43.3 -> 52.8 mm
- net N$6: track 66.1 -> 73.0 mm, vias 2 -> 0
- net N$16: track 20.4 -> 26.3 mm, vias 1 -> 0
- net N$10: track 73.0 -> 68.3 mm, vias 1 -> 0
- net N$22: track 33.5 -> 28.9 mm, vias 1 -> 0
- net N$14: track 25.1 -> 29.7 mm, vias 1 -> 0
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- added copper zone on layer 1, net BUS+
- added copper zone on layer 1, net BUS+2
- added copper zone on layer 16, net BUS+3
Other:
- outline, holes or cut-outs redrawn

Commit message: Плата SP
Parts:
- removed LED1: LAP4-BOTTOM, led:P47F-BOTTOM
- added PWR: (no value), led:CHIPLED_0603
Connections:
- new net N$7: PWR.C
- net N$2: no longer LED1.C
- net N$5: now also PWR.A; no longer LED1.A
Routing:
- added copper zone on layer 1, net BUS+1
- added copper zone on layer 16, net BUS-1
- removed copper zone on layer 1, net BUS+
- removed copper zone on layer 1, net BUS+2
- removed copper zone on layer 16, net BUS+3
Other:
- outline, holes or cut-outs redrawn
Changed lines of the file:
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@@
 <wire x1="23.204940625" y1="28.8618" x2="24.306490625" y2="34.26748125" width="0.1" layer="51" curve="66.964381"/>
 <wire x1="0" y1="0" x2="82" y2="0" width="0.1524" layer="20"/>
-<wire x1="0" y1="82" x2="0" y2="72.25" width="0.1524" layer="20"/>
-<wire x1="0" y1="71.25" x2="0" y2="31.25" width="0.1524" layer="20"/>
-<wire x1="0" y1="30.25" x2="0" y2="0" width="0.1524" layer="20"/>
-<wire x1="82" y1="0" x2="82" y2="9.75" width="0.1524" layer="20"/>
-<wire x1="82" y1="10.75" x2="82" y2="50.75" width="0.1524" layer="20"/>
-<wire x1="82" y1="51.75" x2="82" y2="82" width="0.1524" layer="20"/>
+<wire x1="0" y1="82" x2="0" y2="72.75" width="0.1524" layer="20"/>
+<wire x1="0" y1="70.75" x2="0" y2="31.75" width="0.1524" layer="20"/>
+<wire x1="0" y1="29.75" x2="0" y2="0" width="0.1524" layer="20"/>
+<wire x1="82" y1="0" x2="82" y2="9.25" width="0.1524" layer="20"/>
+<wire x1="82" y1="11.25" x2="82" y2="50.25" width="0.1524" layer="20"/>
+<wire x1="82" y1="52.25" x2="82" y2="82" width="0.1524" layer="20"/>
 <wire x1="82" y1="82" x2="0" y2="82" width="0.1524" layer="20"/>
-<wire x1="82" y1="10.75" x2="81" y2="10.75" width="0.1524" layer="20"/>
+<wire x1="82" y1="11.25" x2="81.5" y2="11.25" width="0.1524" layer="20"/>
+<wire x1="81.5" y1="11.25" x2="81" y2="10.75" width="0.1524" layer="20" curve="90"/>
 <wire x1="81" y1="10.75" x2="81" y2="9.75" width="0.1524" layer="20"/>
-<wire x1="81" y1="9.75" x2="82" y2="9.75" width="0.1524" layer="20"/>
-<wire x1="82" y1="51.75" x2="81" y2="51.75" width="0.1524" layer="20"/>
+<wire x1="81" y1="9.75" x2="81.5" y2="9.25" width="0.1524" layer="20" curve="90"/>
+<wire x1="81.5" y1="9.25" x2="82" y2="9.25" width="0.1524" layer="20"/>
+<wire x1="82" y1="52.25" x2="81.5" y2="52.25" width="0.1524" layer="20"/>
+<wire x1="81.5" y1="52.25" x2="81" y2="51.75" width="0.1524" layer="20" curve="90"/>
 <wire x1="81" y1="51.75" x2="81" y2="50.75" width="0.1524" layer="20"/>
-<wire x1="81" y1="50.75" x2="82" y2="50.75" width="0.1524" layer="20"/>
-<wire x1="0" y1="71.25" x2="1" y2="71.25" width="0.1524" layer="20"/>
+<wire x1="81" y1="50.75" x2="81.5" y2="50.25" width="0.1524" layer="20" curve="90"/>
+<wire x1="81.5" y1="50.25" x2="82" y2="50.25" width="0.1524" layer="20"/>
+<wire x1="0" y1="70.75" x2="0.5" y2="70.75" width="0.1524" layer="20"/>
+<wire x1="0.5" y1="70.75" x2="1" y2="71.25" width="0.1524" layer="20" curve="90"/>
 <wire x1="1" y1="71.25" x2="1" y2="72.25" width="0.1524" layer="20"/>
-<wire x1="1" y1="72.25" x2="0" y2="72.25" width="0.1524" layer="20"/>
-<wire x1="0" y1="30.25" x2="1" y2="30.25" width="0.1524" layer="20"/>
+<wire x1="1" y1="72.25" x2="0.5" y2="72.75" width="0.1524" layer="20" curve="90"/>
+<wire x1="0.5" y1="72.75" x2="0" y2="72.75" width="0.1524" layer="20"/>
+<wire x1="0" y1="29.75" x2="0.5" y2="29.75" width="0.1524" layer="20"/>
+<wire x1="0.5" y1="29.75" x2="1" y2="30.25" width="0.1524" layer="20" curve="90"/>
 <wire x1="1" y1="30.25" x2="1" y2="31.25" width="0.1524" layer="20"/>
-<wire x1="1" y1="31.25" x2="0" y2="31.25" width="0.1524" layer="20"/>
+<wire x1="1" y1="31.25" x2="0.5" y2="31.75" width="0.1524" layer="20" curve="90"/>
+<wire x1="0.5" y1="31.75" x2="0" y2="31.75" width="0.1524" layer="20"/>
 </plain>
 <attributes>
@@
 <attribute name="VALUE" x="21" y="-0.556" size="1.27" layer="28" ratio="10" rot="MR180"/>
 </element>
-<element name="LED1" library="led" library_urn="urn:adsk.eagle:library:259" package="P47F-BOTTOM" package3d_urn="urn:adsk.eagle:package:15878/1" value="LAP4-BOTTOM" x="35.6" y="3" smashed="yes" rot="MR0">
-<attribute name="NAME" x="39.41" y="4.905" size="1.27" layer="26" rot="MR0"/>
-<attribute name="POPULARITY" value="1" x="35.6" y="3" size="1.778" layer="28" rot="MR0" display="off"/>
-<attribute name="VALUE" x="39.41" y="-0.175" size="1.27" layer="28" rot="MR0"/>
-</element>
 <element name="R1" library="rcl" library_urn="urn:adsk.eagle:library:334" package="R0603" package3d_urn="urn:adsk.eagle:package:23555/3" value="2k7" x="37" y="6" smashed="yes" rot="MR180">
 <attribute name="NAME" x="36.365" y="5.365" size="1.27" layer="26" rot="MR180"/>
@@
 <attribute name="SPICEPREFIX" value="R" x="37" y="6" size="1.778" layer="28" rot="MR180" display="off"/>
 <attribute name="VALUE" x="36.365" y="7.905" size="1.27" layer="28" rot="MR180"/>
+</element>
+<element name="PWR" library="led" library_urn="urn:adsk.eagle:library:259" package="CHIPLED_0603" package3d_urn="urn:adsk.eagle:package:15822/2" value="" x="35" y="2.7" smashed="yes" rot="R90">
+<attribute name="NAME" x="36.27" y="2.065" size="1.27" layer="25" rot="R180"/>
+<attribute name="POPULARITY" value="28" x="29.7" y="-2.3" size="1.778" layer="27" rot="R90" display="off"/>
+<attribute name="VALUE" x="36.27" y="4.605" size="1.27" layer="27" rot="R180"/>
 </element>
 </elements>
@@
 <wire x1="16.31" y1="60.9994" x2="16.60355625" y2="61.153803125" width="0.5" layer="1"/>
 <wire x1="16.31" y1="20.8768" x2="16.60355625" y2="20.84619375" width="0.5" layer="1"/>
+<polygon width="0.1524" layer="1" isolate="0.5">
+<vertex x="84.2" y="-1.8"/>
+<vertex x="84.2" y="3"/>
+<vertex x="84.2" y="85.1"/>
+<vertex x="-3.7" y="85.1"/>
+<vertex x="-3.7" y="-1.8"/>
+<vertex x="0.2" y="-1.8"/>
+</polygon>
 </signal>
 <signal name="BUS-1">
@@
 <wire x1="23.4864" y1="3.262" x2="23.5" y2="3" width="0.5" layer="1"/>
 <wire x1="7.1764" y1="10.1122" x2="7" y2="10.25" width="0.5" layer="1"/>
+<polygon width="0.1524" layer="16" isolate="0.5">
+<vertex x="-4.9" y="-2.2"/>
+<vertex x="84.9" y="-2.2"/>
+<vertex x="84.9" y="85.4"/>
+<vertex x="-4.9" y="85.4"/>
+</polygon>
 </signal>
 <signal name="N$4">
@@
 <contactref element="U$19" pad="4"/>
 <contactref element="S1" pad="2"/>
-<contactref element="LED1" pad="C"/>
 <wire x1="24.465" y1="61.6518" x2="29.0318" y2="57.085" width="0.5" layer="1"/>
 <wire x1="29.0318" y1="57.085" x2="29.336196875" y2="56.90644375" width="0.5" layer="1"/>
@@
 <wire x1="20.8768" y1="3.262" x2="23.3233" y2="5.7085" width="0.5" layer="16"/>
 <wire x1="23.3233" y1="5.7085" x2="24.7912" y2="7.1764" width="0.5" layer="16"/>
-<wire x1="32.9462" y1="3.262" x2="33.15" y2="3" width="0.5" layer="16"/>
 <wire x1="20.8768" y1="3.262" x2="21" y2="3" width="0.5" layer="16"/>
 <wire x1="22.1816" y1="19.8982" x2="24.1388" y2="19.8982" width="0.5" layer="16"/>
@@
 </signal>
 <signal name="N$5">
-<contactref element="LED1" pad="A"/>
 <contactref element="R1" pad="1"/>
 <wire x1="38.1654" y1="3.9144" x2="36.2082" y2="5.8716" width="0.5" layer="16"/>
 <wire x1="38.1654" y1="3.262" x2="38.1654" y2="3.9144" width="0.5" layer="16"/>
 <wire x1="36.2082" y1="5.8716" x2="36.15" y2="6" width="0.5" layer="16"/>
-<wire x1="38.1654" y1="3.262" x2="38.05" y2="3" width="0.5" layer="16"/>
-</signal>
-<signal name="BUS+">
-<polygon width="0.1524" layer="1">
-<vertex x="1.25" y="0.25"/>
-<vertex x="80.75" y="0.25"/>
-<vertex x="80.75" y="81.75"/>
-<vertex x="1.25" y="81.75"/>
-</polygon>
-</signal>
-<signal name="BUS+2">
-<polygon width="0.1524" layer="1">
-<vertex x="1.25" y="0.25"/>
-<vertex x="80.75" y="0.25"/>
-<vertex x="80.75" y="81.75"/>
-<vertex x="1.25" y="81.75"/>
-</polygon>
-</signal>
-<signal name="BUS+3">
-<polygon width="0.1524" layer="16">
-<vertex x="1.25" y="0.25"/>
-<vertex x="80.75" y="0.25"/>
-<vertex x="80.75" y="81.75"/>
-<vertex x="1.25" y="81.75"/>
-</polygon>
+<contactref element="PWR" pad="A"/>
+<wire x1="35.75" y1="2.7" x2="36.15" y2="6" width="0" layer="19" extent="1-16"/>
+</signal>
+<signal name="N$7">
+<contactref element="PWR" pad="C"/>
 </signal>
 </signals>
