File: schematics/board/SP.brd (EAGLE design)
At the start: 82 x 82 mm, 44 parts

Commit message: Плата SP
Parts:
- flipped PWR to the bottom, turned to 270 degrees
Connections:
- removed net BUS-1: D29.A, S1.3, SOL1.IN
- removed net N$7: PWR.C
- net N$2: now also D29.A, PWR.C, S1.3, SOL1.IN
Routing:
- net N$2: track 166.7 -> 199.8 mm
- net BUS-1: track 26.5 -> 0.00 mm
- net N$5: track 3.56 -> 3.54 mm, vias 0 -> 1
- added copper zone on layer 16, net N$2
- removed copper zone on layer 16, net BUS-1
Changed lines of the file:
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@@
 <autorouter>
 <pass name="Default">
-<param name="RoutingGrid" value="50mil"/>
+<param name="RoutingGrid" value="0.25mm"/>
 <param name="AutoGrid" value="1"/>
 <param name="Efforts" value="0"/>
 <param name="TopRouterVariant" value="1"/>
 <param name="tpViaShape" value="round"/>
-<param name="PrefDir.1" value="a"/>
+<param name="PrefDir.1" value="-"/>
 <param name="PrefDir.2" value="0"/>
 <param name="PrefDir.3" value="0"/>
@@
 <param name="PrefDir.14" value="0"/>
 <param name="PrefDir.15" value="0"/>
-<param name="PrefDir.16" value="a"/>
+<param name="PrefDir.16" value="|"/>
 <param name="cfVia" value="8"/>
 <param name="cfNonPref" value="5"/>
@@
 <attribute name="VALUE" x="36.365" y="7.905" size="1.27" layer="28" rot="MR180"/>
 </element>
-<element name="PWR" library="led" library_urn="urn:adsk.eagle:library:259" package="CHIPLED_0603" package3d_urn="urn:adsk.eagle:package:15822/2" value="" x="35" y="2.7" smashed="yes" rot="R90">
-<attribute name="NAME" x="36.27" y="2.065" size="1.27" layer="25" rot="R180"/>
-<attribute name="POPULARITY" value="28" x="29.7" y="-2.3" size="1.778" layer="27" rot="R90" display="off"/>
-<attribute name="VALUE" x="36.27" y="4.605" size="1.27" layer="27" rot="R180"/>
+<element name="PWR" library="led" library_urn="urn:adsk.eagle:library:259" package="CHIPLED_0603" package3d_urn="urn:adsk.eagle:package:15822/2" value="" x="35" y="2.7" smashed="yes" rot="MR270">
+<attribute name="NAME" x="36.27" y="3.335" size="1.27" layer="26" rot="MR0"/>
+<attribute name="POPULARITY" value="28" x="29.7" y="7.7" size="1.778" layer="28" rot="MR270" display="off"/>
+<attribute name="VALUE" x="36.27" y="0.795" size="1.27" layer="28" rot="MR0"/>
 </element>
 </elements>
@@
 <contactref element="U$18" pad="1"/>
 <contactref element="U$18" pad="3"/>
-<contactref element="R1" pad="2"/>
 <wire x1="61.3256" y1="65.24" x2="65.24" y2="61.3256" width="0.5" layer="1"/>
 <wire x1="65.24" y1="61.3256" x2="65.396446875" y2="61.153803125" width="0.5" layer="1"/>
@@
 <wire x1="21.5292" y1="17.2886" x2="30.0104" y2="17.2886" width="0.5" layer="16"/>
 <wire x1="20.8768" y1="16.6362" x2="21.5292" y2="17.2886" width="0.5" layer="16"/>
-<wire x1="37.8392" y1="6.1978" x2="37.85" y2="6" width="0.5" layer="16"/>
 <wire x1="20.8768" y1="16.6362" x2="20.846196875" y2="16.603553125" width="0.5" layer="16"/>
 <wire x1="20.5506" y1="16.6362" x2="16.6362" y2="20.5506" width="0.5" layer="1"/>
@@
 <vertex x="0.2" y="-1.8"/>
 </polygon>
-</signal>
-<signal name="BUS-1">
-<contactref element="D29" pad="A"/>
-<contactref element="SOL1" pad="IN"/>
-<contactref element="S1" pad="3"/>
-<wire x1="26.4222" y1="5.8716" x2="29.0318" y2="5.8716" width="0.5" layer="16"/>
-<wire x1="23.8126" y1="3.262" x2="26.4222" y2="5.8716" width="0.5" layer="16"/>
-<wire x1="29.0318" y1="5.8716" x2="29.1" y2="6" width="0.5" layer="16"/>
-<wire x1="23.8126" y1="3.262" x2="23.5" y2="3" width="0.5" layer="16"/>
-<wire x1="16.6362" y1="10.1122" x2="23.4864" y2="3.262" width="0.5" layer="1"/>
-<wire x1="7.1764" y1="10.1122" x2="16.6362" y2="10.1122" width="0.5" layer="1"/>
-<wire x1="23.4864" y1="3.262" x2="23.5" y2="3" width="0.5" layer="1"/>
-<wire x1="7.1764" y1="10.1122" x2="7" y2="10.25" width="0.5" layer="1"/>
-<polygon width="0.1524" layer="16" isolate="0.5">
-<vertex x="-4.9" y="-2.2"/>
-<vertex x="84.9" y="-2.2"/>
-<vertex x="84.9" y="85.4"/>
-<vertex x="-4.9" y="85.4"/>
-</polygon>
+<contactref element="R1" pad="2"/>
+<wire x1="37.75" y1="6" x2="37.85" y2="6" width="0.5" layer="16"/>
+<wire x1="37.75" y1="6" x2="37.8392" y2="6.1978" width="0.5" layer="16"/>
 </signal>
 <signal name="N$4">
@@
 <wire x1="29.0318" y1="24.7912" x2="29.336196875" y2="25.093553125" width="0.5" layer="1"/>
 <wire x1="24.465" y1="20.2244" x2="24.386446875" y2="20.143803125" width="0.5" layer="1"/>
-<wire x1="32.9462" y1="3.9144" x2="32.9462" y2="3.262" width="0.5" layer="16"/>
-<wire x1="30.3366" y1="6.524" x2="32.9462" y2="3.9144" width="0.5" layer="16"/>
-<wire x1="30.3366" y1="6.8502" x2="30.3366" y2="6.524" width="0.5" layer="16"/>
-<wire x1="30.0104" y1="7.1764" x2="30.3366" y2="6.8502" width="0.5" layer="16"/>
-<wire x1="24.7912" y1="7.1764" x2="30.0104" y2="7.1764" width="0.5" layer="16"/>
 <wire x1="20.8768" y1="3.262" x2="23.3233" y2="5.7085" width="0.5" layer="16"/>
-<wire x1="23.3233" y1="5.7085" x2="24.7912" y2="7.1764" width="0.5" layer="16"/>
 <wire x1="20.8768" y1="3.262" x2="21" y2="3" width="0.5" layer="16"/>
 <wire x1="22.1816" y1="19.8982" x2="24.1388" y2="19.8982" width="0.5" layer="16"/>
@@
 <wire x1="50.561" y1="31.3152" x2="51.5396" y2="32.2938" width="0.5" layer="1"/>
 <wire x1="50.561" y1="25.1174" x2="50.561" y2="31.3152" width="0.5" layer="1"/>
+<contactref element="PWR" pad="C"/>
+<wire x1="32.5" y1="11.5" x2="32.5" y2="4.5" width="0.5" layer="1"/>
+<wire x1="24.5" y1="19.5" x2="32.5" y2="11.5" width="0.5" layer="1"/>
+<wire x1="24.5" y1="20" x2="24.5" y2="19.5" width="0.5" layer="1"/>
+<wire x1="24.5" y1="20" x2="24.386446875" y2="20.143803125" width="0.5" layer="1"/>
+<contactref element="D29" pad="A"/>
+<contactref element="SOL1" pad="IN"/>
+<contactref element="S1" pad="3"/>
+<wire x1="26.4222" y1="5.8716" x2="29.0318" y2="5.8716" width="0.5" layer="16"/>
+<wire x1="23.8126" y1="3.262" x2="26.4222" y2="5.8716" width="0.5" layer="16"/>
+<wire x1="29.0318" y1="5.8716" x2="29.1" y2="6" width="0.5" layer="16"/>
+<wire x1="23.8126" y1="3.262" x2="23.5" y2="3" width="0.5" layer="16"/>
+<wire x1="16.6362" y1="10.1122" x2="23.4864" y2="3.262" width="0.5" layer="1"/>
+<wire x1="7.1764" y1="10.1122" x2="16.6362" y2="10.1122" width="0.5" layer="1"/>
+<wire x1="23.4864" y1="3.262" x2="23.5" y2="3" width="0.5" layer="1"/>
+<wire x1="7.1764" y1="10.1122" x2="7" y2="10.25" width="0.5" layer="1"/>
+<polygon width="0.1524" layer="16" isolate="0.5">
+<vertex x="-4.9" y="-2.2"/>
+<vertex x="84.9" y="-2.2"/>
+<vertex x="84.9" y="85.4"/>
+<vertex x="-4.9" y="85.4"/>
+</polygon>
 </signal>
 <signal name="N$5">
 <contactref element="R1" pad="1"/>
-<wire x1="38.1654" y1="3.9144" x2="36.2082" y2="5.8716" width="0.5" layer="16"/>
-<wire x1="38.1654" y1="3.262" x2="38.1654" y2="3.9144" width="0.5" layer="16"/>
-<wire x1="36.2082" y1="5.8716" x2="36.15" y2="6" width="0.5" layer="16"/>
 <contactref element="PWR" pad="A"/>
-<wire x1="35.75" y1="2.7" x2="36.15" y2="6" width="0" layer="19" extent="1-16"/>
-</signal>
-<signal name="N$7">
-<contactref element="PWR" pad="C"/>
+<wire x1="36" y1="6" x2="36" y2="4.5" width="0.5" layer="16"/>
+<via x="36" y="4.5" extent="1-16" drill="0.35"/>
+<wire x1="36" y1="6" x2="36.15" y2="6" width="0.5" layer="16"/>
+<wire x1="36" y1="4.5" x2="36" y2="3" width="0.5" layer="16"/>
+<wire x1="36" y1="3" x2="35.75" y2="2.7" width="0.5" layer="16"/>
 </signal>
 </signals>

Commit message: Плата SPv2
Connections:
- new net BUS-1: D29.A, S1.3, SOL1.IN
- net N$2: no longer D29.A, S1.3, SOL1.IN
Routing:
- net N$2: track 199.8 -> 175.1 mm, vias 0 -> 1
- net BUS-1: track 0.00 -> 16.9 mm, vias 0 -> 1
- net N$5: vias 1 -> 0
- added copper zone on layer 16, net BUS-1
- removed copper zone on layer 16, net N$2
Changed lines of the file:
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@@
 <vertex x="-3.7" y="85.1"/>
 <vertex x="-3.7" y="-1.8"/>
-<vertex x="0.2" y="-1.8"/>
 </polygon>
 <contactref element="R1" pad="2"/>
@@
 <wire x1="29.0318" y1="24.7912" x2="29.336196875" y2="25.093553125" width="0.5" layer="1"/>
 <wire x1="24.465" y1="20.2244" x2="24.386446875" y2="20.143803125" width="0.5" layer="1"/>
-<wire x1="20.8768" y1="3.262" x2="23.3233" y2="5.7085" width="0.5" layer="16"/>
-<wire x1="20.8768" y1="3.262" x2="21" y2="3" width="0.5" layer="16"/>
 <wire x1="22.1816" y1="19.8982" x2="24.1388" y2="19.8982" width="0.5" layer="16"/>
 <wire x1="19.572" y1="17.2886" x2="22.1816" y2="19.8982" width="0.5" layer="16"/>
 <wire x1="19.572" y1="9.4598" x2="19.572" y2="17.2886" width="0.5" layer="16"/>
-<wire x1="23.3233" y1="5.7085" x2="19.572" y2="9.4598" width="0.5" layer="16"/>
+<wire x1="22.5159" y1="6.5159" x2="19.572" y2="9.4598" width="0.5" layer="16"/>
 <wire x1="24.1388" y1="19.8982" x2="24.386446875" y2="20.143803125" width="0.5" layer="16"/>
 <wire x1="29.358" y1="25.1174" x2="50.561" y2="25.1174" width="0.5" layer="1"/>
@@
 <wire x1="24.5" y1="20" x2="24.5" y2="19.5" width="0.5" layer="1"/>
 <wire x1="24.5" y1="20" x2="24.386446875" y2="20.143803125" width="0.5" layer="1"/>
-<contactref element="D29" pad="A"/>
-<contactref element="SOL1" pad="IN"/>
-<contactref element="S1" pad="3"/>
-<wire x1="26.4222" y1="5.8716" x2="29.0318" y2="5.8716" width="0.5" layer="16"/>
-<wire x1="23.8126" y1="3.262" x2="26.4222" y2="5.8716" width="0.5" layer="16"/>
-<wire x1="29.0318" y1="5.8716" x2="29.1" y2="6" width="0.5" layer="16"/>
-<wire x1="23.8126" y1="3.262" x2="23.5" y2="3" width="0.5" layer="16"/>
-<wire x1="16.6362" y1="10.1122" x2="23.4864" y2="3.262" width="0.5" layer="1"/>
-<wire x1="7.1764" y1="10.1122" x2="16.6362" y2="10.1122" width="0.5" layer="1"/>
-<wire x1="23.4864" y1="3.262" x2="23.5" y2="3" width="0.5" layer="1"/>
-<wire x1="7.1764" y1="10.1122" x2="7" y2="10.25" width="0.5" layer="1"/>
-<polygon width="0.1524" layer="16" isolate="0.5">
-<vertex x="-4.9" y="-2.2"/>
-<vertex x="84.9" y="-2.2"/>
-<vertex x="84.9" y="85.4"/>
-<vertex x="-4.9" y="85.4"/>
-</polygon>
+<wire x1="32.5" y1="4.5" x2="34" y2="3" width="0.5" layer="16"/>
+<wire x1="34" y1="3" x2="34.25" y2="2.7" width="0.5" layer="16"/>
+<wire x1="21" y1="5" x2="22.5159" y2="6.5159" width="0.5" layer="16"/>
+<wire x1="21" y1="3" x2="21" y2="5" width="0.5" layer="16"/>
+<via x="32.5" y="4.5" extent="1-16" drill="0.35"/>
 </signal>
 <signal name="N$5">
 <contactref element="R1" pad="1"/>
 <contactref element="PWR" pad="A"/>
-<wire x1="36" y1="6" x2="36" y2="4.5" width="0.5" layer="16"/>
-<via x="36" y="4.5" extent="1-16" drill="0.35"/>
+<wire x1="36" y1="6" x2="36" y2="3" width="0.5" layer="16"/>
+<wire x1="36" y1="3" x2="35.75" y2="2.7" width="0.5" layer="16"/>
 <wire x1="36" y1="6" x2="36.15" y2="6" width="0.5" layer="16"/>
-<wire x1="36" y1="4.5" x2="36" y2="3" width="0.5" layer="16"/>
-<wire x1="36" y1="3" x2="35.75" y2="2.7" width="0.5" layer="16"/>
+</signal>
+<signal name="BUS-1">
+<contactref element="D29" pad="A"/>
+<contactref element="SOL1" pad="IN"/>
+<contactref element="S1" pad="3"/>
+<wire x1="26.4" y1="5.8716" x2="26.5" y2="5.8716" width="0.5" layer="16"/>
+<wire x1="26.5" y1="5.8716" x2="29.0318" y2="5.8716" width="0.5" layer="16"/>
+<wire x1="29.0318" y1="5.8716" x2="29.1" y2="6" width="0.5" layer="16"/>
+<wire x1="7.1764" y1="10.1122" x2="12" y2="10.1122" width="0.5" layer="1"/>
+<wire x1="12" y1="10.1122" x2="16.6362" y2="10.1122" width="0.5" layer="1"/>
+<wire x1="7.1764" y1="10.1122" x2="7" y2="10.25" width="0.5" layer="1"/>
+<wire x1="23.5" y1="3" x2="26.5" y2="6" width="0.5" layer="16"/>
+<wire x1="26.5" y1="6" x2="26.5" y2="5.8716" width="0.5" layer="16"/>
+<polygon width="0.5" layer="16" isolate="0.5">
+<vertex x="-5.4" y="89.8"/>
+<vertex x="-5.4" y="-3.7"/>
+<vertex x="86" y="-3.7"/>
+<vertex x="86" y="89.8"/>
+</polygon>
+<wire x1="12" y1="10" x2="12" y2="10.1122" width="0.5" layer="1"/>
+<via x="12" y="10" extent="1-16" drill="0.35"/>
 </signal>
 </signals>

Commit message: Плата SPv3
Routing:
- net BUS-1: track 16.9 -> 30.5 mm
- net N$2: track 175.1 -> 172.6 mm
- added copper zone on layer 16, net N$2
- removed copper zone on layer 16, net BUS-1
Changed lines of the file:
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@@
 <wire x1="24.5" y1="20" x2="24.5" y2="19.5" width="0.5" layer="1"/>
 <wire x1="24.5" y1="20" x2="24.386446875" y2="20.143803125" width="0.5" layer="1"/>
-<wire x1="32.5" y1="4.5" x2="34" y2="3" width="0.5" layer="16"/>
-<wire x1="34" y1="3" x2="34.25" y2="2.7" width="0.5" layer="16"/>
 <wire x1="21" y1="5" x2="22.5159" y2="6.5159" width="0.5" layer="16"/>
 <wire x1="21" y1="3" x2="21" y2="5" width="0.5" layer="16"/>
 <via x="32.5" y="4.5" extent="1-16" drill="0.35"/>
+<polygon width="0.5" layer="16">
+<vertex x="-14.1" y="-8.2"/>
+<vertex x="89.7" y="-8.2"/>
+<vertex x="89.7" y="91.3"/>
+<vertex x="-14.1" y="91.3"/>
+</polygon>
 </signal>
 <signal name="N$5">
@@
 <contactref element="SOL1" pad="IN"/>
 <contactref element="S1" pad="3"/>
-<wire x1="26.4" y1="5.8716" x2="26.5" y2="5.8716" width="0.5" layer="16"/>
-<wire x1="26.5" y1="5.8716" x2="29.0318" y2="5.8716" width="0.5" layer="16"/>
 <wire x1="29.0318" y1="5.8716" x2="29.1" y2="6" width="0.5" layer="16"/>
 <wire x1="7.1764" y1="10.1122" x2="12" y2="10.1122" width="0.5" layer="1"/>
-<wire x1="12" y1="10.1122" x2="16.6362" y2="10.1122" width="0.5" layer="1"/>
+<wire x1="12" y1="10.1122" x2="15" y2="10.1122" width="0.5" layer="1"/>
 <wire x1="7.1764" y1="10.1122" x2="7" y2="10.25" width="0.5" layer="1"/>
-<wire x1="23.5" y1="3" x2="26.5" y2="6" width="0.5" layer="16"/>
-<wire x1="26.5" y1="6" x2="26.5" y2="5.8716" width="0.5" layer="16"/>
-<polygon width="0.5" layer="16" isolate="0.5">
-<vertex x="-5.4" y="89.8"/>
-<vertex x="-5.4" y="-3.7"/>
-<vertex x="86" y="-3.7"/>
-<vertex x="86" y="89.8"/>
-</polygon>
 <wire x1="12" y1="10" x2="12" y2="10.1122" width="0.5" layer="1"/>
 <via x="12" y="10" extent="1-16" drill="0.35"/>
+<wire x1="23.5" y1="7.5" x2="23.5" y2="3" width="0.5" layer="1"/>
+<wire x1="17.5" y1="7.5" x2="23.5" y2="7.5" width="0.5" layer="1"/>
+<wire x1="15" y1="10" x2="17.5" y2="7.5" width="0.5" layer="1"/>
+<wire x1="15" y1="10" x2="15" y2="10.1122" width="0.5" layer="1"/>
+<wire x1="24.5" y1="6" x2="29.1" y2="6" width="0.5" layer="16"/>
+<wire x1="24.5" y1="4.5" x2="24.5" y2="6" width="0.5" layer="16"/>
+<wire x1="23.5" y1="3.5" x2="24.5" y2="4.5" width="0.5" layer="16"/>
+<wire x1="23.5" y1="3" x2="23.5" y2="3.5" width="0.5" layer="16"/>
 </signal>
 </signals>
