File: schematics/board/TESTPL.sch (EAGLE design)
At the start: 31 parts

Commit message: Исправлена плата TESTPL
Parts:
- removed LED-G: (no value), led:LEDCHIPLED_0603
- added JP20, JP21, JP22, JP23, JP24, JP25, JP26, JP27, JP28, JP29, JP30, JP31: (no value), pinheadCS:PINHD-1X1
- added JP32: (no value), pinheadCS:PINHD-1X2
- added LED, LED-G1, LED-G10, LED-G11, LED-G12, LED-G2, LED-G3, LED-G4, LED-G5, LED-G6, LED-G7, LED-G8, LED-G9: (no value), led:LEDCHIPLED_0603
- added R1, R2, R3, R4, R5, R7: R100, rcl:R-US_R2512
- added R10, R11, R12, R13, R14, R15, R16, R17, R18, R19, R8, R9: 2k7, resistor:R-US_R0603
- U$1: value 6.8R -> 6R8
- U$2: value 0.68R -> R68
- U$4: value 1.1R -> 1R1
- U$5, U$6: value 2.2R -> 2R2
- U$7: value 3.9R -> 3R9
- U$8: value 4.7R -> 4R7
Connections:
- new net GND: JP21.1, JP23.1, JP25.1, JP27.1, JP29.1, JP3.1, JP31.1, JP4.1, LED.C, R1.1, R2.1, R3.1, R4.1, R5.1, R7.1, U$1.2
- new net N$12: JP19.1, JP28.1, LED-G11.A, LED-G5.C, R5.2
- new net N$13: JP18.1, JP26.1, LED-G10.A, LED-G4.C, R4.2
- new net N$14: JP14.1, JP24.1, LED-G3.C, LED-G9.A, R3.2
- new net N$15: JP15.1, JP22.1, LED-G2.C, LED-G8.A, R2.2
- new net N$16: JP16.1, JP20.1, LED-G1.C, LED-G7.A, R1.2
- new net N$17: JP13.1, JP32.2, R6.1, U$10.1
- new net N$18: LED-G1.A, R8.2
- new net N$19: LED-G2.A, R9.2
- new net N$20: LED-G3.A, R10.2
- new net N$21: LED-G4.A, R11.2
- new net N$22: LED-G5.A, R12.2
- new net N$23: LED-G6.A, R13.2
- new net N$24: LED-G8.C, R15.1
- new net N$25: LED-G7.C, R14.1
- new net N$26: LED-G9.C, R16.1
- new net N$27: LED-G10.C, R17.1
- new net N$28: LED-G11.C, R18.1
- new net N$29: LED-G12.C, R19.1
- net N$10: now also JP30.1, LED-G12.A, LED-G6.C, R7.2; no longer JP14.1, JP15.1, JP16.1, JP18.1, JP19.1, JP3.1, JP4.1, LED-G.C, U$1.2
- net N$11: now also JP32.1, R10.1, R11.1, R12.1, R13.1, R14.2, R15.2, R16.2, R17.2, R18.2, R19.2, R8.1, R9.1; no longer JP13.1, R6.1, U$10.1
- net N$38: now also LED.A; no longer LED-G.A
Other:
- moved on the sheet: JP14, JP15, JP16, JP17, JP18, JP19, JP2, R6
