File: schematics/board/MAG.sch (EAGLE design)
At the start: 12 parts

Commit message: Платы подготовлены для Резонита
Parts:
- renumbered JP2 to GND, JP3 to 3V3, JP4 to SDA, JP5 to SCL
Changed lines of the file:
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@@
 <?xml version="1.0" encoding="utf-8"?>
 <!DOCTYPE eagle SYSTEM "eagle.dtd">
-<eagle version="9.6.0">
+<eagle version="9.4.2">
 <drawing>
 <settings>
@@
 <part name="C10" library="rcl" library_urn="urn:adsk.eagle:library:334" deviceset="C-US" device="C0603" package3d_urn="urn:adsk.eagle:package:23616/2" value="0,1µ"/>
 <part name="C1" library="rcl" library_urn="urn:adsk.eagle:library:334" deviceset="C-US" device="C0603" package3d_urn="urn:adsk.eagle:package:23616/2" value="0,1µ"/>
-<part name="JP2" library="pinheadCS" deviceset="PINHD-1X1" device=""/>
-<part name="JP3" library="pinheadCS" deviceset="PINHD-1X1" device=""/>
-<part name="JP4" library="pinheadCS" deviceset="PINHD-1X1" device=""/>
-<part name="JP5" library="pinheadCS" deviceset="PINHD-1X1" device=""/>
+<part name="GND" library="pinheadCS" deviceset="PINHD-1X1" device=""/>
+<part name="3V3" library="pinheadCS" deviceset="PINHD-1X1" device=""/>
+<part name="SDA" library="pinheadCS" deviceset="PINHD-1X1" device=""/>
+<part name="SCL" library="pinheadCS" deviceset="PINHD-1X1" device=""/>
 <part name="R101" library="resistor" library_urn="urn:adsk.eagle:library:348" deviceset="R-US_" device="R0603" package3d_urn="urn:adsk.eagle:package:23555/3" value="5k1"/>
 <part name="R102" library="resistor" library_urn="urn:adsk.eagle:library:348" deviceset="R-US_" device="R0603" package3d_urn="urn:adsk.eagle:package:23555/3" value="5k1"/>
@@
 <attribute name="VALUE" x="34.036" y="21.209" size="1.778" layer="96"/>
 </instance>
-<instance part="JP2" gate="G$1" x="-5.08" y="-38.1" smashed="yes" rot="R270">
+<instance part="GND" gate="G$1" x="-5.08" y="-38.1" smashed="yes" rot="R270">
 <attribute name="NAME" x="-1.905" y="-31.75" size="1.778" layer="95" rot="R270"/>
 <attribute name="VALUE" x="-10.16" y="-31.75" size="1.778" layer="96" rot="R270"/>
 </instance>
-<instance part="JP3" gate="G$1" x="5.08" y="-38.1" smashed="yes" rot="R270">
+<instance part="3V3" gate="G$1" x="5.08" y="-38.1" smashed="yes" rot="R270">
 <attribute name="NAME" x="8.255" y="-31.75" size="1.778" layer="95" rot="R270"/>
 <attribute name="VALUE" x="0" y="-31.75" size="1.778" layer="96" rot="R270"/>
 </instance>
-<instance part="JP4" gate="G$1" x="15.24" y="-38.1" smashed="yes" rot="R270">
+<instance part="SDA" gate="G$1" x="15.24" y="-38.1" smashed="yes" rot="R270">
 <attribute name="NAME" x="18.415" y="-31.75" size="1.778" layer="95" rot="R270"/>
 <attribute name="VALUE" x="10.16" y="-31.75" size="1.778" layer="96" rot="R270"/>
 </instance>
-<instance part="JP5" gate="G$1" x="25.4" y="-38.1" smashed="yes" rot="R270">
+<instance part="SCL" gate="G$1" x="25.4" y="-38.1" smashed="yes" rot="R270">
 <attribute name="NAME" x="28.575" y="-31.75" size="1.778" layer="95" rot="R270"/>
 <attribute name="VALUE" x="20.32" y="-31.75" size="1.778" layer="96" rot="R270"/>
@@
 <wire x1="5.08" y1="-35.56" x2="5.08" y2="-22.86" width="0.1524" layer="91"/>
 <label x="5.08" y="-27.94" size="1.778" layer="95" rot="R90"/>
-<pinref part="JP3" gate="G$1" pin="1"/>
+<pinref part="3V3" gate="G$1" pin="1"/>
 </segment>
 <segment>
@@
 <pinref part="R1" gate="G$1" pin="1"/>
 <wire x1="-7.62" y1="-20.32" x2="-5.08" y2="-20.32" width="0.1524" layer="91"/>
-<pinref part="JP2" gate="G$1" pin="1"/>
+<pinref part="GND" gate="G$1" pin="1"/>
 </segment>
 <segment>
@@
 <label x="15.24" y="-27.94" size="1.778" layer="95" rot="R90"/>
 <pinref part="R102" gate="G$1" pin="2"/>
-<pinref part="JP4" gate="G$1" pin="1"/>
+<pinref part="SDA" gate="G$1" pin="1"/>
 </segment>
 </net>
@@
 <label x="25.4" y="-27.94" size="1.778" layer="95" rot="R90"/>
 <pinref part="R101" gate="G$1" pin="2"/>
-<pinref part="JP5" gate="G$1" pin="1"/>
-</segment>
-</net>
+<pinref part="SCL" gate="G$1" pin="1"/>
+</segment>
+</net>

Commit message: Исправлены MAG и BSK1
Connections:
- net N$1: now also PWR.C; no longer PWR.A
- net VDD: now also PWR.A; no longer PWR.C
Other:
- moved on the sheet: PWR
Changed lines of the file:
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@@
 <part name="LIS3MDL" library="CanCubeSat" deviceset="LIS3MDL" device=""/>
 <part name="LSM6DS3" library="CanCubeSat" deviceset="LSM6DS3" device=""/>
-<part name="PWR" library="led" library_urn="urn:adsk.eagle:library:259" deviceset="LED" device="CHIPLED_0603" package3d_urn="urn:adsk.eagle:package:15822/2"/>
 <part name="R1" library="resistor" library_urn="urn:adsk.eagle:library:348" deviceset="R-US_" device="R0603" package3d_urn="urn:adsk.eagle:package:23555/3" value="2k"/>
 <part name="C10" library="rcl" library_urn="urn:adsk.eagle:library:334" deviceset="C-US" device="C0603" package3d_urn="urn:adsk.eagle:package:23616/2" value="0,1µ"/>
@@
 <part name="R101" library="resistor" library_urn="urn:adsk.eagle:library:348" deviceset="R-US_" device="R0603" package3d_urn="urn:adsk.eagle:package:23555/3" value="5k1"/>
 <part name="R102" library="resistor" library_urn="urn:adsk.eagle:library:348" deviceset="R-US_" device="R0603" package3d_urn="urn:adsk.eagle:package:23555/3" value="5k1"/>
+<part name="PWR" library="led" library_urn="urn:adsk.eagle:library:259" deviceset="LED" device="CHIPLED_0603" package3d_urn="urn:adsk.eagle:package:15822/2"/>
 </parts>
 <sheets>
@@
 <attribute name="NAME" x="45.72" y="53.34" size="2.1844" layer="95"/>
 </instance>
-<instance part="PWR" gate="G$1" x="-20.32" y="-20.32" smashed="yes" rot="R270">
-<attribute name="NAME" x="-24.892" y="-23.876" size="1.778" layer="95"/>
-<attribute name="VALUE" x="-24.892" y="-26.035" size="1.778" layer="96"/>
-</instance>
 <instance part="R1" gate="G$1" x="-12.7" y="-20.32" smashed="yes" rot="R180">
 <attribute name="NAME" x="-8.89" y="-21.8186" size="1.778" layer="95" rot="R180"/>
@@
 <attribute name="NAME" x="16.7386" y="-8.89" size="1.778" layer="95" rot="R270"/>
 <attribute name="VALUE" x="11.938" y="-8.89" size="1.778" layer="96" rot="R270"/>
+</instance>
+<instance part="PWR" gate="G$1" x="-22.86" y="-20.32" smashed="yes" rot="R90">
+<attribute name="NAME" x="-18.288" y="-16.764" size="1.778" layer="95" rot="R180"/>
+<attribute name="VALUE" x="-18.288" y="-14.605" size="1.778" layer="96" rot="R180"/>
 </instance>
 </instances>
@@
 </busses>
 <nets>
-<net name="N$1" class="0">
-<segment>
-<pinref part="R1" gate="G$1" pin="2"/>
-<pinref part="PWR" gate="G$1" pin="A"/>
-</segment>
-</net>
 <net name="VDD" class="0">
 <segment>
-<pinref part="PWR" gate="G$1" pin="C"/>
 <wire x1="-25.4" y1="-20.32" x2="-33.02" y2="-20.32" width="0.1524" layer="91"/>
 <label x="-33.02" y="-20.32" size="1.778" layer="95"/>
+<pinref part="PWR" gate="G$1" pin="A"/>
 </segment>
 <segment>
@@
 </segment>
 </net>
+<net name="N$1" class="0">
+<segment>
+<pinref part="PWR" gate="G$1" pin="C"/>
+<pinref part="R1" gate="G$1" pin="2"/>
+</segment>
+</net>

Commit message: Исправлена плата MAG
Changed lines of the file:
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@@
 <layers>
 <layer number="1" name="Top" color="4" fill="1" visible="no" active="no"/>
+<layer number="2" name="Route2" color="16" fill="1" visible="no" active="no"/>
+<layer number="3" name="Route3" color="17" fill="1" visible="no" active="no"/>
+<layer number="4" name="Route4" color="18" fill="1" visible="no" active="no"/>
+<layer number="5" name="Route5" color="19" fill="1" visible="no" active="no"/>
+<layer number="6" name="Route6" color="25" fill="1" visible="no" active="no"/>
+<layer number="7" name="Route7" color="26" fill="1" visible="no" active="no"/>
+<layer number="8" name="Route8" color="27" fill="1" visible="no" active="no"/>
+<layer number="9" name="Route9" color="28" fill="1" visible="no" active="no"/>
+<layer number="10" name="Route10" color="29" fill="1" visible="no" active="no"/>
+<layer number="11" name="Route11" color="30" fill="1" visible="no" active="no"/>
+<layer number="12" name="Route12" color="20" fill="1" visible="no" active="no"/>
+<layer number="13" name="Route13" color="21" fill="1" visible="no" active="no"/>
+<layer number="14" name="Route14" color="22" fill="1" visible="no" active="no"/>
+<layer number="15" name="Route15" color="23" fill="1" visible="no" active="no"/>
 <layer number="16" name="Bottom" color="1" fill="1" visible="no" active="no"/>
 <layer number="17" name="Pads" color="2" fill="1" visible="no" active="no"/>
@@
 <layer number="48" name="Document" color="7" fill="1" visible="no" active="no"/>
 <layer number="49" name="Reference" color="7" fill="1" visible="no" active="no"/>
+<layer number="50" name="dxf" color="7" fill="1" visible="no" active="no"/>
 <layer number="51" name="tDocu" color="7" fill="1" visible="no" active="no"/>
 <layer number="52" name="bDocu" color="7" fill="1" visible="no" active="no"/>
+<layer number="53" name="tGND_GNDA" color="7" fill="9" visible="no" active="no"/>
+<layer number="54" name="bGND_GNDA" color="1" fill="9" visible="no" active="no"/>
+<layer number="56" name="wert" color="7" fill="1" visible="no" active="no"/>
 <layer number="88" name="SimResults" color="9" fill="1" visible="yes" active="yes"/>
 <layer number="89" name="SimProbes" color="9" fill="1" visible="yes" active="yes"/>
@@
 <layer number="101" name="NotChangedData" color="15" fill="1" visible="yes" active="yes"/>
 <layer number="102" name="ChangedData" color="15" fill="1" visible="yes" active="yes"/>
+<layer number="103" name="tMap" color="7" fill="1" visible="no" active="no"/>
+<layer number="104" name="Name" color="7" fill="1" visible="no" active="no"/>
+<layer number="105" name="tPlate" color="7" fill="1" visible="no" active="no"/>
+<layer number="106" name="bPlate" color="7" fill="1" visible="no" active="no"/>
+<layer number="107" name="Crop" color="7" fill="1" visible="no" active="no"/>
+<layer number="108" name="fp8" color="7" fill="1" visible="no" active="no"/>
+<layer number="109" name="fp9" color="7" fill="1" visible="no" active="no"/>
+<layer number="110" name="110" color="7" fill="1" visible="no" active="no"/>
+<layer number="111" name="111" color="7" fill="1" visible="no" active="no"/>
+<layer number="112" name="tSilk" color="7" fill="1" visible="no" active="no"/>
+<layer number="113" name="IDFDebug" color="7" fill="1" visible="no" active="yes"/>
+<layer number="116" name="Patch_BOT" color="9" fill="4" visible="no" active="no"/>
+<layer number="118" name="Rect_Pads" color="7" fill="1" visible="no" active="no"/>
+<layer number="121" name="_tsilk" color="7" fill="1" visible="no" active="no"/>
+<layer number="122" name="_bsilk" color="7" fill="1" visible="no" active="no"/>
+<layer number="123" name="tTestmark" color="7" fill="1" visible="no" active="no"/>
+<layer number="124" name="bTestmark" color="7" fill="1" visible="no" active="no"/>
+<layer number="125" name="_tNames" color="7" fill="1" visible="no" active="no"/>
+<layer number="126" name="_bNames" color="7" fill="1" visible="no" active="no"/>
+<layer number="127" name="_tValues" color="7" fill="1" visible="no" active="no"/>
+<layer number="128" name="_bValues" color="7" fill="1" visible="no" active="no"/>
+<layer number="131" name="tAdjust" color="7" fill="1" visible="no" active="no"/>
+<layer number="132" name="bAdjust" color="7" fill="1" visible="no" active="no"/>
+<layer number="144" name="DrillLegend" color="7" fill="1" visible="no" active="no"/>
+<layer number="151" name="HeatSink" color="14" fill="1" visible="no" active="no"/>
+<layer number="152" name="_bDocu" color="7" fill="1" visible="no" active="no"/>
+<layer number="199" name="Contour" color="7" fill="1" visible="no" active="no"/>
+<layer number="200" name="200bmp" color="1" fill="10" visible="no" active="no"/>
+<layer number="201" name="201bmp" color="2" fill="1" visible="no" active="no"/>
+<layer number="202" name="202bmp" color="3" fill="1" visible="no" active="no"/>
+<layer number="203" name="203bmp" color="4" fill="10" visible="no" active="no"/>
+<layer number="204" name="204bmp" color="5" fill="10" visible="no" active="no"/>
+<layer number="205" name="205bmp" color="6" fill="10" visible="no" active="no"/>
+<layer number="206" name="206bmp" color="7" fill="10" visible="no" active="no"/>
+<layer number="207" name="207bmp" color="15" fill="10" visible="no" active="no"/>
+<layer number="208" name="208bmp" color="9" fill="10" visible="no" active="no"/>
+<layer number="209" name="209bmp" color="7" fill="1" visible="no" active="no"/>
+<layer number="210" name="210bmp" color="7" fill="1" visible="no" active="no"/>
+<layer number="211" name="211bmp" color="7" fill="1" visible="no" active="no"/>
+<layer number="212" name="212bmp" color="7" fill="1" visible="no" active="no"/>
+<layer number="213" name="213bmp" color="7" fill="1" visible="no" active="no"/>
+<layer number="214" name="214bmp" color="7" fill="1" visible="no" active="no"/>
+<layer number="215" name="215bmp" color="7" fill="1" visible="no" active="no"/>
+<layer number="216" name="216bmp" color="7" fill="1" visible="no" active="no"/>
+<layer number="217" name="217bmp" color="18" fill="1" visible="no" active="no"/>
+<layer number="218" name="218bmp" color="19" fill="1" visible="no" active="no"/>
+<layer number="219" name="219bmp" color="20" fill="1" visible="no" active="no"/>
+<layer number="220" name="220bmp" color="21" fill="1" visible="no" active="no"/>
+<layer number="221" name="221bmp" color="22" fill="1" visible="no" active="no"/>
+<layer number="222" name="222bmp" color="23" fill="1" visible="no" active="no"/>
+<layer number="223" name="223bmp" color="24" fill="1" visible="no" active="no"/>
+<layer number="224" name="224bmp" color="25" fill="1" visible="no" active="no"/>
+<layer number="225" name="225bmp" color="7" fill="1" visible="no" active="yes"/>
+<layer number="226" name="226bmp" color="7" fill="1" visible="no" active="yes"/>
+<layer number="227" name="227bmp" color="7" fill="1" visible="no" active="yes"/>
+<layer number="228" name="228bmp" color="7" fill="1" visible="no" active="yes"/>
+<layer number="230" name="230bmp" color="7" fill="1" visible="no" active="yes"/>
+<layer number="248" name="Housing" color="7" fill="1" visible="no" active="no"/>
+<layer number="249" name="Edge" color="7" fill="1" visible="no" active="no"/>
+<layer number="250" name="Descript" color="3" fill="1" visible="no" active="no"/>
+<layer number="251" name="SMDround" color="12" fill="11" visible="no" active="no"/>
+<layer number="254" name="OrgLBR" color="13" fill="1" visible="no" active="no"/>
 </layers>
 <schematic xreflabel="%F%N/%S.%C%R" xrefpart="/%S.%C%R">
