File: schematics/Debug/Debug.sch (EAGLE design)
At the start: 11 parts

Commit message: Кнопка на отладочной плате
Parts:
- added S1: (no value), switch-omron:10-XX
Connections:
- removed net GND: JP3.1, JP6.1, JP8.1, JP9.1
- removed net N$14: JP1.1, JP1.2, JP1.3, JP1.4, JP1.5, JP1.6, U$1.GND
- new net N$10: JP1.1, JP1.2, JP1.3, JP1.4, JP1.5, JP1.6, JP3.1, JP6.2, JP8.1, JP9.3, S1.P, S1.P1, U$1.GND
- net N$11: now also U$1.SWDIO; no longer U$1.SWDC
- net N$12: now also JP9.1, U$1.SWDC; no longer JP9.3, U$1.SWDIO
- net N$4: now also S1.S, S1.S1
- net N$6: now also JP6.1; no longer JP6.2
Other:
- moved on the sheet: JP1, JP2, JP3, JP5, JP6, JP7, JP9, R1, R2

Commit message: Debug plata
Parts:
- R1, R2: device resistor:R-EU_0204/5 -> rcl:R-EU_R0603
- renumbered JP1 to GND, JP2 to RADIO_M1, JP3 to BUS1, JP5 to U_STM32, JP6 to BUS0, JP7 to U_ESP32, JP8 to RESET, JP9 to SWD/UART
Connections:
- net N$10 renamed GND
- net N$6 renamed BUS
- net N$9 renamed M1
- removed net N$1: U$1.TX-, U_STM32.2
- removed net N$11: SWD/UART.2, U$1.SWDIO
- removed net N$12: SWD/UART.1, U$1.SWDC
- removed net N$2: U$1.RX-, U_STM32.1
- removed net N$3: U$1.RX+, U_ESP32.1
- removed net N$4: RESET.2, S1.S, S1.S1, U$1.SBU1
- removed net N$5: U$1.TX+, U_ESP32.2
- new net RESET: RESET.2, S1.S, S1.S1, U$1.RES
- new net RX+: U$1.RX1, U_ESP32.1
- new net RX-: U$1.RX0, U_STM32.1
- new net SWC: SWD/UART.1, U$1.SWC
- new net SWD: SWD/UART.2, U$1.SWD
- new net TX+: U$1.TX1, U_ESP32.2
- new net TX-: U$1.TX0, U_STM32.2
Other:
- moved on the sheet: R1, R2

Commit message: Очередная дебажная плата
Parts:
- removed BUS0, U_ESP32, U_STM32: (no value), pinhead:PINHD-1X2
- removed GND: (no value), pinhead:PINHD-1X6
- removed SWD/UART: (no value), pinhead:PINHD-1X3
- added BUS2, BUS3, BUS4, DB_ESP, DB_STM, IO0, RESET1: (no value), pinhead:PINHD-1X2
- added DL_ESP, DL_STM: (no value), pinhead:PINHD-1X3
- added GND1: (no value), pinhead:PINHD-1X6
- added S2, S3: (no value), switch-omron:10-XX
- added U$2: USB-C, CanCubeSat:USB-C
Connections:
- removed net RX+: U$1.RX1, U_ESP32.1
- removed net RX-: U$1.RX0, U_STM32.1
- removed net SWC: SWD/UART.1, U$1.SWC
- removed net SWD: SWD/UART.2, U$1.SWD
- removed net TX+: U$1.TX1, U_ESP32.2
- removed net TX-: U$1.TX0, U_STM32.2
- new net 3V3: BUS2.2, BUS3.2, U$1.NC, U$2.NC
- new net N$3: IO0.1, S3.P, S3.P1, U$1.IO0
- new net RESET_STM: RESET1.2, S2.S, S2.S1, U$2.RES
- new net RX0: DB_ESP.1, U$1.RX0
- new net RX0_STM: DB_STM.1, U$2.RX0
- new net RX1: DL_ESP.2, U$1.RX1/SWD
- new net SWC_STM: DL_STM.3, U$2.TX1/SWC
- new net SWD_STM: DL_STM.2, U$2.RX1/SWD
- new net TX0: DB_ESP.2, U$1.TX0
- new net TX0_STM: DB_STM.2, U$2.TX0
- new net TX1: DL_ESP.3, U$1.TX1/SWC
- net BUS: now also BUS4.2, U$2.VBUS; no longer BUS0.1
- net GND: now also BUS2.1, BUS3.1, BUS4.1, DL_STM.1, GND1.1, GND1.2, GND1.3, GND1.4, GND1.5, GND1.6, IO0.2, RESET1.1, S2.P, S2.P1, S3.S, S3.S1, U$2.GND; no longer BUS0.2, GND.1, GND.2, GND.3, GND.4, GND.5, GND.6, SWD/UART.3
Other:
- note added: "ESP32"
- note added: "STM32"
- moved on the sheet: BUS1, R1, R2, RADIO_M1, RESET, S1

Commit message: Отладочная плата v2
Parts:
- removed BUS1, BUS2, BUS3, BUS4, DB_ESP, DB_STM, RADIO_M1, RESET, RESET1: (no value), pinhead:PINHD-1X2
- removed DL_ESP, DL_STM: (no value), pinhead:PINHD-1X3
- removed GND1: (no value), pinhead:PINHD-1X6
- removed R1: 1k, rcl:R-EU_R0603
- removed R2: 10k, rcl:R-EU_R0603
- removed S1, S2, S3: (no value), switch-omron:10-XX
- added C1, C2, C3: 1nF, rcl:C-USC0603
- added DEBUG_STM32: (no value), pinhead:PINHD-1X3
- added DOWNLOAD_ESP32: (no value), pinhead:PINHD-1X5
- added DOWNLOAD_STM32, RADIO: (no value), pinhead:PINHD-1X4
- added EN, NRST: (no value), switch-omron:10-XX
- added ENABLE, GPIO0, JP1, JP5, JP6, JP7, JP8, NRESET: (no value), pinhead:PINHD-1X2
- added JP2: (no value), pinhead:PINHD-1X6
- IO0: device pinhead:PINHD-1X2 -> switch-omron:10-XX
Connections:
- removed net N$3: IO0.1, S3.P, S3.P1, U$1.IO0
- removed net N$7: R1.2, RADIO_M1.1
- removed net N$8: R1.1, R2.1
- removed net RESET: RESET.2, S1.S, S1.S1, U$1.RES
- removed net RESET_STM: RESET1.2, S2.S, S2.S1, U$2.RES
- removed net RX0: DB_ESP.1, U$1.RX0
- removed net RX0_STM: DB_STM.1, U$2.RX0
- removed net SWC_STM: DL_STM.3, U$2.TX1/SWC
- removed net SWD_STM: DL_STM.2, U$2.RX1/SWD
- removed net TX0: DB_ESP.2, U$1.TX0
- removed net TX0_STM: DB_STM.2, U$2.TX0
- new net 3V3-S: JP1.1, U$1.NC/3V3
- new net EN: C2.2, DOWNLOAD_ESP32.5, EN.P, EN.P1, ENABLE.2, U$1.NRST/EN
- new net IO0: C1.2, DOWNLOAD_ESP32.4, GPIO0.2, IO0.P, IO0.P1, U$1.NC/GPIO
- new net NRST: C3.2, DOWNLOAD_STM32.4, NRESET.2, NRST.P, NRST.P1, U$2.NRST/EN
- new net RX: DEBUG_STM32.3, U$2.RX0
- new net RXD: DOWNLOAD_ESP32.3, U$1.SWD/RXD
- new net SWC: DOWNLOAD_STM32.2, U$2.SWC/TXD
- new net SWD: DOWNLOAD_STM32.3, U$2.SWD/RXD
- new net TX: DEBUG_STM32.2, U$2.TX0
- new net TXD: DOWNLOAD_ESP32.2, U$1.SWC/TXD
- net 3V3: now also JP5.2, JP7.2, U$2.NC/3V3; no longer BUS2.2, BUS3.2, U$1.NC, U$2.NC
- net BUS: now also JP6.2, JP8.2, U$1.3V3/BUS, U$2.3V3/BUS; no longer BUS1.2, BUS4.2, R2.2, U$1.VBUS, U$2.VBUS
- net GND: now also C1.1, C2.1, C3.1, DEBUG_STM32.1, DOWNLOAD_ESP32.1, DOWNLOAD_STM32.1, EN.S, EN.S1, ENABLE.1, GPIO0.1, IO0.S, IO0.S1, JP2.1, JP2.2, JP2.3, JP2.4, JP2.5, JP2.6, JP5.1, JP6.1, JP7.1, JP8.1, NRESET.1, NRST.S, NRST.S1, RADIO.1; no longer BUS1.1, BUS2.1, BUS3.1, BUS4.1, DL_STM.1, GND1.1, GND1.2, GND1.3, GND1.4, GND1.5, GND1.6, IO0.2, RESET.1, RESET1.1, S1.P, S1.P1, S2.P, S2.P1, S3.S, S3.S1
- net M1: now also JP1.2, RADIO.4, U$1.NC/M1; no longer RADIO_M1.2, U$1.M1
- net RX1: now also RADIO.3, U$1.RX0; no longer DL_ESP.2, U$1.RX1/SWD
- net TX1: now also RADIO.2, U$1.TX0; no longer DL_ESP.3, U$1.TX1/SWC

Commit message: Отладочная плата v3
Connections:
- net 3V3: now also U$2.3V3/BUS; no longer U$2.NC/3V3
- net BUS: no longer U$2.3V3/BUS
Changed lines of the file:
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@@
 <wire x1="175.26" y1="66.04" x2="175.26" y2="53.34" width="0.1524" layer="91"/>
 <junction x="182.88" y="66.04"/>
-<pinref part="U$2" gate="G$1" pin="3V3/BUS"/>
-<wire x1="119.38" y1="66.04" x2="114.3" y2="66.04" width="0.1524" layer="91"/>
-<wire x1="175.26" y1="53.34" x2="114.3" y2="53.34" width="0.1524" layer="91"/>
-<wire x1="114.3" y1="53.34" x2="114.3" y2="66.04" width="0.1524" layer="91"/>
 <label x="165.1" y="53.34" size="1.778" layer="95"/>
-<junction x="114.3" y="53.34"/>
 <pinref part="U$1" gate="G$1" pin="3V3/BUS"/>
 <wire x1="30.48" y1="66.04" x2="25.4" y2="66.04" width="0.1524" layer="91"/>
-<wire x1="114.3" y1="53.34" x2="25.4" y2="53.34" width="0.1524" layer="91"/>
+<wire x1="175.26" y1="53.34" x2="25.4" y2="53.34" width="0.1524" layer="91"/>
 <wire x1="25.4" y1="53.34" x2="25.4" y2="66.04" width="0.1524" layer="91"/>
 </segment>
@@
 <pinref part="JP7" gate="G$1" pin="2"/>
 <wire x1="193.04" y1="55.88" x2="182.88" y2="55.88" width="0.1524" layer="91"/>
-<pinref part="U$2" gate="G$1" pin="NC/3V3"/>
-<wire x1="119.38" y1="63.5" x2="116.84" y2="63.5" width="0.1524" layer="91"/>
-<wire x1="182.88" y1="55.88" x2="116.84" y2="55.88" width="0.1524" layer="91"/>
-<wire x1="116.84" y1="55.88" x2="116.84" y2="63.5" width="0.1524" layer="91"/>
+<wire x1="182.88" y1="55.88" x2="114.3" y2="55.88" width="0.1524" layer="91"/>
 <junction x="182.88" y="55.88"/>
 <label x="165.1" y="55.88" size="1.778" layer="95"/>
+<wire x1="114.3" y1="55.88" x2="114.3" y2="66.04" width="0.1524" layer="91"/>
+<pinref part="U$2" gate="G$1" pin="3V3/BUS"/>
+<wire x1="114.3" y1="66.04" x2="119.38" y2="66.04" width="0.1524" layer="91"/>
 </segment>
 </net>

Commit message: Логическая схема для сбросом и управление бутлоадером ESP32 на отладочной плате.
Parts:
- added R1, R2: 10, rcl:R-EU_R0603
- added T1, T2: 2n7002, zetex:NMOSSOT23
Connections:
- new net DTR: DOWNLOAD_ESP32.5, R1.1, T2.S
- new net N$1: R2.2, T2.G
- new net N$2: R1.2, T1.G
- new net RTS: DOWNLOAD_ESP32.4, R2.1, T1.S
- net EN: now also T1.D; no longer DOWNLOAD_ESP32.5
- net IO0: now also T2.D; no longer DOWNLOAD_ESP32.4
Other:
- note added: "Auto program DTR RTS -> EN IO0 1 1 1 1 0 0 1 1 1 0 0 1 0 1 1 0"
- moved on the sheet: DOWNLOAD_ESP32

Commit message: Внёс незначительные правки на платах. Но пока не везде
Parts:
- added 3V3, 8V: (no value), led:LEDCHIPLED_0603
- added R3, R4: 2k, rcl:R-EU_R0603
Connections:
- new net N$3: 3V3.C, R4.2
- new net N$4: 8V.C, R3.2
- net 3V3: now also 3V3.A
- net BUS: now also 8V.A
- net GND: now also R3.1, R4.1
Changed lines of the file:
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@@
 <?xml version="1.0" encoding="utf-8"?>
 <!DOCTYPE eagle SYSTEM "eagle.dtd">
-<eagle version="9.5.2">
+<eagle version="9.5.1">
 <drawing>
 <settings>
@@
 <layer number="98" name="Guide" color="6" fill="1" visible="yes" active="yes"/>
 <layer number="99" name="SpiceOrder" color="5" fill="1" visible="no" active="no"/>
+<layer number="100" name="DocFrame" color="15" fill="1" visible="yes" active="yes"/>
+<layer number="101" name="NotChangedData" color="15" fill="1" visible="yes" active="yes"/>
+<layer number="102" name="ChangedData" color="15" fill="1" visible="yes" active="yes"/>
 </layers>
 <schematic xreflabel="%F%N/%S.%C%R" xrefpart="/%S.%C%R">
@@
 <part name="R1" library="rcl" library_urn="urn:adsk.eagle:library:334" deviceset="R-EU_" device="R0603" package3d_urn="urn:adsk.eagle:package:23555/3" value="10"/>
 <part name="R2" library="rcl" library_urn="urn:adsk.eagle:library:334" deviceset="R-EU_" device="R0603" package3d_urn="urn:adsk.eagle:package:23555/3" value="10"/>
+<part name="R3" library="rcl" library_urn="urn:adsk.eagle:library:334" deviceset="R-EU_" device="R0603" package3d_urn="urn:adsk.eagle:package:23555/3" value="2k"/>
+<part name="R4" library="rcl" library_urn="urn:adsk.eagle:library:334" deviceset="R-EU_" device="R0603" package3d_urn="urn:adsk.eagle:package:23555/3" value="2k"/>
+<part name="8V" library="led" library_urn="urn:adsk.eagle:library:259" deviceset="LED" device="CHIPLED_0603" package3d_urn="urn:adsk.eagle:package:15822/2"/>
+<part name="3V3" library="led" library_urn="urn:adsk.eagle:library:259" deviceset="LED" device="CHIPLED_0603" package3d_urn="urn:adsk.eagle:package:15822/2"/>
 </parts>
 <sheets>
@@
 <attribute name="NAME" x="-6.35" y="-41.6814" size="1.778" layer="95"/>
 <attribute name="VALUE" x="-6.35" y="-46.482" size="1.778" layer="96"/>
+</instance>
+<instance part="R3" gate="G$1" x="203.2" y="71.12" smashed="yes">
+<attribute name="NAME" x="199.39" y="72.6186" size="1.778" layer="95"/>
+<attribute name="VALUE" x="199.39" y="67.818" size="1.778" layer="96"/>
+</instance>
+<instance part="R4" gate="G$1" x="203.2" y="58.42" smashed="yes">
+<attribute name="NAME" x="199.39" y="59.9186" size="1.778" layer="95"/>
+<attribute name="VALUE" x="199.39" y="55.118" size="1.778" layer="96"/>
+</instance>
+<instance part="8V" gate="G$1" x="213.36" y="71.12" smashed="yes" rot="R270">
+<attribute name="NAME" x="208.788" y="67.564" size="1.778" layer="95"/>
+<attribute name="VALUE" x="208.788" y="65.405" size="1.778" layer="96"/>
+</instance>
+<instance part="3V3" gate="G$1" x="213.36" y="58.42" smashed="yes" rot="R270">
+<attribute name="NAME" x="208.788" y="54.864" size="1.778" layer="95"/>
+<attribute name="VALUE" x="208.788" y="52.705" size="1.778" layer="96"/>
 </instance>
 </instances>
@@
 <junction x="55.88" y="43.18"/>
 <label x="55.88" y="-71.12" size="1.778" layer="95" rot="R90"/>
+<pinref part="R3" gate="G$1" pin="1"/>
+<junction x="193.04" y="68.58"/>
+<pinref part="R4" gate="G$1" pin="1"/>
+<wire x1="198.12" y1="58.42" x2="193.04" y2="58.42" width="0.1524" layer="91"/>
+<junction x="193.04" y="58.42"/>
+<wire x1="193.04" y1="68.58" x2="198.12" y2="68.58" width="0.1524" layer="91"/>
+<wire x1="198.12" y1="68.58" x2="198.12" y2="71.12" width="0.1524" layer="91"/>
 </segment>
 </net>
@@
 <wire x1="175.26" y1="53.34" x2="25.4" y2="53.34" width="0.1524" layer="91"/>
 <wire x1="25.4" y1="53.34" x2="25.4" y2="66.04" width="0.1524" layer="91"/>
+<pinref part="8V" gate="G$1" pin="A"/>
+<wire x1="215.9" y1="71.12" x2="218.44" y2="71.12" width="0.1524" layer="91"/>
+<wire x1="218.44" y1="71.12" x2="218.44" y2="66.04" width="0.1524" layer="91"/>
+<wire x1="218.44" y1="66.04" x2="193.04" y2="66.04" width="0.1524" layer="91"/>
+<junction x="193.04" y="66.04"/>
 </segment>
 </net>
@@
 <pinref part="U$2" gate="G$1" pin="3V3/BUS"/>
 <wire x1="114.3" y1="66.04" x2="119.38" y2="66.04" width="0.1524" layer="91"/>
+<pinref part="3V3" gate="G$1" pin="A"/>
+<wire x1="215.9" y1="58.42" x2="218.44" y2="58.42" width="0.1524" layer="91"/>
+<wire x1="218.44" y1="58.42" x2="218.44" y2="53.34" width="0.1524" layer="91"/>
+<wire x1="218.44" y1="53.34" x2="198.12" y2="53.34" width="0.1524" layer="91"/>
+<wire x1="198.12" y1="53.34" x2="198.12" y2="55.88" width="0.1524" layer="91"/>
+<wire x1="198.12" y1="55.88" x2="193.04" y2="55.88" width="0.1524" layer="91"/>
+<junction x="193.04" y="55.88"/>
 </segment>
 </net>
@@
 </segment>
 </net>
+<net name="N$3" class="0">
+<segment>
+<pinref part="3V3" gate="G$1" pin="C"/>
+<pinref part="R4" gate="G$1" pin="2"/>
+</segment>
+</net>
+<net name="N$4" class="0">
+<segment>
+<pinref part="R3" gate="G$1" pin="2"/>
+<pinref part="8V" gate="G$1" pin="C"/>
+</segment>
+</net>

Commit message: Подписал контакты, отправил плату в производство
Parts:
- renumbered 3V3 to LED1, 8V to LED2
